File: demos/sonde xilinx/sonde xilinx.sch (KiCad schematic (older format))
At the start: 25 parts, among them J1 DB25MALE, J2 DB9MALE, P1 CONN_6, U1 74LS125, U2 74LS125

Commit message: Update demos
Parts:
- C1: symbol CP -> sonde~xilinx_schlib:CP
- C2, C3, C4, C5: symbol C -> sonde~xilinx_schlib:C
- D1, D2: symbol DIODESCH -> sonde~xilinx_schlib:DIODESCH
- J1: symbol DB25 -> sonde~xilinx_schlib:DB25
- J2: symbol DB9 -> sonde~xilinx_schlib:DB9
- P1: symbol CONN_6 -> sonde~xilinx_schlib:CONN_6
- R1, R10, R11, R12, R13, R14, R2, R4, R5, R6, R7, R8, R9: symbol R -> sonde~xilinx_schlib:R
- U1, U2: symbol 74LS125 -> sonde~xilinx_schlib:74LS125
Changed lines of the file:
@@
-EESchema Schematic File Version 2
-LIBS:sonde xilinx_schlib
-LIBS:power
+EESchema Schematic File Version 4
 LIBS:sonde xilinx-cache
-EELAYER 25 0
+EELAYER 26 0
 EELAYER END
 $Descr A4 11693 8268
@@
 $EndDescr
 $Comp
-L R R11
+L sonde~xilinx_schlib:R R11
 U 1 1 4D527316
 P 6650 2600
@@
 	5900 4200 6400 4200
 $Comp
-L GND #PWR01
+L sonde~xilinx_schlib:GND #PWR01
 U 1 1 3EBF81B1
 P 6300 4700
@@
 $EndComp
 $Comp
-L C C4
+L sonde~xilinx_schlib:C C4
 U 1 1 3EBF81A7
 P 6300 4450
@@
 $EndComp
 $Comp
-L R R13
+L sonde~xilinx_schlib:R R13
 U 1 1 4D528082
 P 6650 4200
@@
 	4800 4500 5450 4500
 $Comp
-L 74LS125 U1
+L sonde~xilinx_schlib:74LS125 U1
 U 4 1 3EBF7DBD
 P 5450 4200
@@
 	10200 4200 10250 4200
 $Comp
-L DB9 J2
+L sonde~xilinx_schlib:DB9 J2
 U 1 1 3ECDE5C8
 P 10700 3900
@@
 	8400 3700 8400 2750
 $Comp
-L PWR_FLAG #FLG02
+L sonde~xilinx_schlib:PWR_FLAG #FLG02
 U 1 1 3EBF848F
 P 6100 950
@@
 $EndComp
 $Comp
-L VCC #PWR03
+L sonde~xilinx_schlib:VCC #PWR03
 U 1 1 3EBF8479
 P 5800 950
@@
 $EndComp
 $Comp
-L GND #PWR04
+L sonde~xilinx_schlib:GND #PWR04
 U 1 1 3EBF8458
 P 10200 4850
@@
 $EndComp
 $Comp
-L PWR_FLAG #FLG05
+L sonde~xilinx_schlib:PWR_FLAG #FLG05
 U 1 1 3EBF843C
 P 10200 4800
@@
 	2500 2700 2200 2700
 $Comp
-L GND #PWR06
+L sonde~xilinx_schlib:GND #PWR06
 U 1 1 4D528081
 P 2500 2750
@@
 PWR_3,3-5V
 $Comp
-L GND #PWR07
+L sonde~xilinx_schlib:GND #PWR07
 U 1 1 4D52808A
 P 10050 3600
@@
 PWR_3,3-5V
 $Comp
-L GND #PWR08
+L sonde~xilinx_schlib:GND #PWR08
 U 1 1 3EBF8376
 P 8450 2650
@@
 	7300 1000 9400 1000
 $Comp
-L CONN_6 P1
+L sonde~xilinx_schlib:CONN_6 P1
 U 1 1 3EBF830C
 P 8850 2800
@@
 	6500 1000 6500 1050
 $Comp
-L GND #PWR09
+L sonde~xilinx_schlib:GND #PWR09
 U 1 1 3EBF82CF
 P 6500 1500
@@
 $EndComp
 $Comp
-L CP C1
+L sonde~xilinx_schlib:CP C1
 U 1 1 3EBF82C6
 P 6500 1250
@@
 	5850 1900 6400 1900
 $Comp
-L GND #PWR010
+L sonde~xilinx_schlib:GND #PWR010
 U 1 1 4D528089
 P 6300 3800
@@
 $EndComp
 $Comp
-L C C5
+L sonde~xilinx_schlib:C C5
 U 1 1 4D528086
 P 6300 3550
@@
 $EndComp
 $Comp
-L R R12
+L sonde~xilinx_schlib:R R12
 U 1 1 4D528083
 P 6650 3300
@@
 $EndComp
 $Comp
-L GND #PWR011
+L sonde~xilinx_schlib:GND #PWR011
 U 1 1 4D528088
 P 6300 3100
@@
 $EndComp
 $Comp
-L C C2
+L sonde~xilinx_schlib:C C2
 U 1 1 4D528085
 P 6300 2850
@@
 	6200 1000 6200 1050
 $Comp
-L GND #PWR012
+L sonde~xilinx_schlib:GND #PWR012
 U 1 1 3EBF81B3
 P 6200 1600
@@
 $EndComp
 $Comp
-L GND #PWR013
+L sonde~xilinx_schlib:GND #PWR013
 U 1 1 4D528087
 P 6300 2400
@@
 $EndComp
 $Comp
-L C C3
+L sonde~xilinx_schlib:C C3
 U 1 1 4D528084
 P 6300 2150
@@
 $EndComp
 $Comp
-L R R14
+L sonde~xilinx_schlib:R R14
 U 1 1 3EBF819B
 P 6650 1900
@@
 $EndComp
 $Comp
-L R R5
+L sonde~xilinx_schlib:R R5
 U 1 1 3EBF818E
 P 6200 1300
@@
 $EndComp
 $Comp
-L R R2
+L sonde~xilinx_schlib:R R2
 U 1 1 3EBF8187
 P 5900 1300
@@
 $EndComp
 $Comp
-L DIODESCH D2
+L sonde~xilinx_schlib:DIODESCH D2
 U 1 1 3EBF8176
 P 7100 1000
@@
 $EndComp
 $Comp
-L DIODESCH D1
+L sonde~xilinx_schlib:DIODESCH D1
 U 1 1 3EBF815E
 P 4500 1000
@@
 	2500 1700 2200 1700
 $Comp
-L GND #PWR014
+L sonde~xilinx_schlib:GND #PWR014
 U 1 1 3EBF8100
 P 2500 1750
@@
 $EndComp
 $Comp
-L GND #PWR015
+L sonde~xilinx_schlib:GND #PWR015
 U 1 1 3EBF80DD
 P 4650 2000
@@
 	1150 7200 1700 7200
 $Comp
-L GND #PWR016
+L sonde~xilinx_schlib:GND #PWR016
 U 1 1 3EBF7F0D
 P 1150 7300
@@
 	1150 5600 1250 5600
 $Comp
-L 74LS125 U2
+L sonde~xilinx_schlib:74LS125 U2
 U 4 1 3EBF7EEC
 P 1700 5600
@@
 $EndComp
 $Comp
-L 74LS125 U2
+L sonde~xilinx_schlib:74LS125 U2
 U 3 1 3EBF7EDF
 P 1700 6250
@@
 $EndComp
 $Comp
-L 74LS125 U2
+L sonde~xilinx_schlib:74LS125 U2
 U 2 1 3EBF7EDD
 P 1700 6900
@@
 	4650 2000 4650 1900
 $Comp
-L 74LS125 U1
+L sonde~xilinx_schlib:74LS125 U1
 U 3 1 3EBF7DB3
 P 5450 3300
@@
 $EndComp
 $Comp
-L 74LS125 U1
+L sonde~xilinx_schlib:74LS125 U1
 U 2 1 3EBF7DAD
 P 5450 2600
@@
 $EndComp
 $Comp
-L 74LS125 U1
+L sonde~xilinx_schlib:74LS125 U1
 U 1 1 3EBF7D9F
 P 5400 1900
@@
 $EndComp
 $Comp
-L 74LS125 U2
+L sonde~xilinx_schlib:74LS125 U2
 U 1 1 3EBF7D92
 P 4650 1600
@@
 	2200 1600 3700 1600
 $Comp
-L R R9
+L sonde~xilinx_schlib:R R9
 U 1 1 3EBF7D33
 P 3950 4200
@@
 $EndComp
 $Comp
-L R R10
+L sonde~xilinx_schlib:R R10
 U 1 1 3EBF7D31
 P 3950 3300
@@
 $EndComp
 $Comp
-L R R8
+L sonde~xilinx_schlib:R R8
 U 1 1 4D528080
 P 3950 2900
@@
 $EndComp
 $Comp
-L R R7
+L sonde~xilinx_schlib:R R7
 U 1 1 4D52807F
 P 3950 2600
@@
 $EndComp
 $Comp
-L R R6
+L sonde~xilinx_schlib:R R6
 U 1 1 3EBF7D26
 P 3950 2250
@@
 $EndComp
 $Comp
-L R R4
+L sonde~xilinx_schlib:R R4
 U 1 1 3EBF7D22
 P 3950 1600
@@
 $EndComp
 $Comp
-L R R1
+L sonde~xilinx_schlib:R R1
 U 1 1 3EBF7D16
 P 3950 1000
@@
 $EndComp
 $Comp
-L DB25 J1
+L sonde~xilinx_schlib:DB25 J1
 U 1 1 3EBF7D04
 P 1750 2800
@@
 Connection ~ 7650 1000
 $Comp
-L GND #PWR017
+L sonde~xilinx_schlib:GND #PWR017
 U 1 1 5510FC05
 P 4950 2000

Commit message: Update demo
Parts:
- C1: footprint Discret:CP5 -> Capacitor_THT:C_Axial_L5.1mm_D3.1mm_P12.50mm_Horizontal
- C2, C3, C4, C5: footprint Discret:C2 -> Capacitor_THT:C_Disc_D5.1mm_W3.2mm_P5.00mm
- D1, D2: footprint Discret:D3 -> Diode_THT:D_A-405_P7.62mm_Horizontal
- R1, R10, R11, R12, R13, R14, R2, R4, R5, R6, R7, R8, R9: footprint Discret:R4 -> Resistor_THT:R_Axial_DIN0207_L6.3mm_D2.5mm_P10.16mm_Horizontal
- U1, U2: footprint Sockets_DIP:DIP-14__300_ELL -> Package_DIP:DIP-14_W7.62mm_LongPads

Commit message: Update demos
Parts:
- C1: symbol sonde~xilinx_schlib:CP -> sonde_xilinx_schlib:CP
- C2, C3, C4, C5: symbol sonde~xilinx_schlib:C -> sonde_xilinx_schlib:C
- D1, D2: symbol sonde~xilinx_schlib:DIODESCH -> sonde_xilinx_schlib:DIODESCH
- J1: symbol sonde~xilinx_schlib:DB25 -> sonde_xilinx_schlib:DB25
- J2: symbol sonde~xilinx_schlib:DB9 -> sonde_xilinx_schlib:DB9
- P1: footprint Connect:bornier6 -> Connector_PinHeader_2.54mm:PinHeader_1x06_P2.54mm_Vertical; symbol sonde~xilinx_schlib:CONN_6 -> sonde_xilinx_schlib:CONN_6
- R1, R10, R11, R12, R13, R14, R2, R4, R5, R6, R7, R8, R9: symbol sonde~xilinx_schlib:R -> sonde_xilinx_schlib:R
- U1, U2: symbol sonde~xilinx_schlib:74LS125 -> sonde_xilinx_schlib:74LS125
Changed lines of the file:
@@
 $EndDescr
 $Comp
-L sonde~xilinx_schlib:R R11
+L sonde_xilinx_schlib:R R11
 U 1 1 4D527316
 P 6650 2600
@@
 	5900 4200 6300 4200
 $Comp
-L sonde~xilinx_schlib:GND #PWR01
+L sonde_xilinx_schlib:GND #PWR01
 U 1 1 3EBF81B1
 P 6300 4700
@@
 $EndComp
 $Comp
-L sonde~xilinx_schlib:C C4
+L sonde_xilinx_schlib:C C4
 U 1 1 3EBF81A7
 P 6300 4450
@@
 $EndComp
 $Comp
-L sonde~xilinx_schlib:R R13
+L sonde_xilinx_schlib:R R13
 U 1 1 4D528082
 P 6650 4200
@@
 	4800 4500 5450 4500
 $Comp
-L sonde~xilinx_schlib:74LS125 U1
+L sonde_xilinx_schlib:74LS125 U1
 U 4 1 3EBF7DBD
 P 5450 4200
@@
 	10200 4200 10250 4200
 $Comp
-L sonde~xilinx_schlib:DB9 J2
+L sonde_xilinx_schlib:DB9 J2
 U 1 1 3ECDE5C8
 P 10700 3900
@@
 	8400 3700 8400 2750
 $Comp
-L sonde~xilinx_schlib:PWR_FLAG #FLG02
+L sonde_xilinx_schlib:PWR_FLAG #FLG02
 U 1 1 3EBF848F
 P 6100 950
@@
 $EndComp
 $Comp
-L sonde~xilinx_schlib:VCC #PWR03
+L sonde_xilinx_schlib:VCC #PWR03
 U 1 1 3EBF8479
 P 5800 950
@@
 $EndComp
 $Comp
-L sonde~xilinx_schlib:GND #PWR04
+L sonde_xilinx_schlib:GND #PWR04
 U 1 1 3EBF8458
 P 10200 4850
@@
 $EndComp
 $Comp
-L sonde~xilinx_schlib:PWR_FLAG #FLG05
+L sonde_xilinx_schlib:PWR_FLAG #FLG05
 U 1 1 3EBF843C
 P 10200 4800
@@
 	2500 2700 2200 2700
 $Comp
-L sonde~xilinx_schlib:GND #PWR06
+L sonde_xilinx_schlib:GND #PWR06
 U 1 1 4D528081
 P 2500 2750
@@
 PWR_3,3-5V
 $Comp
-L sonde~xilinx_schlib:GND #PWR07
+L sonde_xilinx_schlib:GND #PWR07
 U 1 1 4D52808A
 P 10050 3600
@@
 PWR_3,3-5V
 $Comp
-L sonde~xilinx_schlib:GND #PWR08
+L sonde_xilinx_schlib:GND #PWR08
 U 1 1 3EBF8376
 P 8450 2650
@@
 	7300 1000 7650 1000
 $Comp
-L sonde~xilinx_schlib:CONN_6 P1
+L sonde_xilinx_schlib:CONN_6 P1
 U 1 1 3EBF830C
 P 8850 2800
 F 0 "P1" V 8800 2800 60  0000 C CNN
 F 1 "CONN_6" V 8900 2800 60  0000 C CNN
-F 2 "Connect:bornier6" H 8850 2800 60  0001 C CNN
+F 2 "Connector_PinHeader_2.54mm:PinHeader_1x06_P2.54mm_Vertical" H 8850 2800 60  0001 C CNN
 F 3 "" H 8850 2800 60  0001 C CNN
 	1    8850 2800
@@
 	6500 1000 6500 1050
 $Comp
-L sonde~xilinx_schlib:GND #PWR09
+L sonde_xilinx_schlib:GND #PWR09
 U 1 1 3EBF82CF
 P 6500 1500
@@
 $EndComp
 $Comp
-L sonde~xilinx_schlib:CP C1
+L sonde_xilinx_schlib:CP C1
 U 1 1 3EBF82C6
 P 6500 1250
@@
 	5850 1900 5900 1900
 $Comp
-L sonde~xilinx_schlib:GND #PWR010
+L sonde_xilinx_schlib:GND #PWR010
 U 1 1 4D528089
 P 6300 3800
@@
 $EndComp
 $Comp
-L sonde~xilinx_schlib:C C5
+L sonde_xilinx_schlib:C C5
 U 1 1 4D528086
 P 6300 3550
@@
 $EndComp
 $Comp
-L sonde~xilinx_schlib:R R12
+L sonde_xilinx_schlib:R R12
 U 1 1 4D528083
 P 6650 3300
@@
 $EndComp
 $Comp
-L sonde~xilinx_schlib:GND #PWR011
+L sonde_xilinx_schlib:GND #PWR011
 U 1 1 4D528088
 P 6300 3100
@@
 $EndComp
 $Comp
-L sonde~xilinx_schlib:C C2
+L sonde_xilinx_schlib:C C2
 U 1 1 4D528085
 P 6300 2850
@@
 	6200 1000 6200 1050
 $Comp
-L sonde~xilinx_schlib:GND #PWR012
+L sonde_xilinx_schlib:GND #PWR012
 U 1 1 3EBF81B3
 P 6200 1600
@@
 $EndComp
 $Comp
-L sonde~xilinx_schlib:GND #PWR013
+L sonde_xilinx_schlib:GND #PWR013
 U 1 1 4D528087
 P 6300 2400
@@
 $EndComp
 $Comp
-L sonde~xilinx_schlib:C C3
+L sonde_xilinx_schlib:C C3
 U 1 1 4D528084
 P 6300 2150
@@
 $EndComp
 $Comp
-L sonde~xilinx_schlib:R R14
+L sonde_xilinx_schlib:R R14
 U 1 1 3EBF819B
 P 6650 1900
@@
 $EndComp
 $Comp
-L sonde~xilinx_schlib:R R5
+L sonde_xilinx_schlib:R R5
 U 1 1 3EBF818E
 P 6200 1300
@@
 $EndComp
 $Comp
-L sonde~xilinx_schlib:R R2
+L sonde_xilinx_schlib:R R2
 U 1 1 3EBF8187
 P 5900 1300
@@
 $EndComp
 $Comp
-L sonde~xilinx_schlib:DIODESCH D2
+L sonde_xilinx_schlib:DIODESCH D2
 U 1 1 3EBF8176
 P 7100 1000
@@
 $EndComp
 $Comp
-L sonde~xilinx_schlib:DIODESCH D1
+L sonde_xilinx_schlib:DIODESCH D1
 U 1 1 3EBF815E
 P 4500 1000
@@
 	2500 1700 2200 1700
 $Comp
-L sonde~xilinx_schlib:GND #PWR014
+L sonde_xilinx_schlib:GND #PWR014
 U 1 1 3EBF8100
 P 2500 1750
@@
 $EndComp
 $Comp
-L sonde~xilinx_schlib:GND #PWR015
+L sonde_xilinx_schlib:GND #PWR015
 U 1 1 3EBF80DD
 P 4650 2000
@@
 	1150 7200 1700 7200
 $Comp
-L sonde~xilinx_schlib:GND #PWR016
+L sonde_xilinx_schlib:GND #PWR016
 U 1 1 3EBF7F0D
 P 1150 7300
@@
 	1150 5600 1250 5600
 $Comp
-L sonde~xilinx_schlib:74LS125 U2
+L sonde_xilinx_schlib:74LS125 U2
 U 4 1 3EBF7EEC
 P 1700 5600
@@
 $EndComp
 $Comp
-L sonde~xilinx_schlib:74LS125 U2
+L sonde_xilinx_schlib:74LS125 U2
 U 3 1 3EBF7EDF
 P 1700 6250
@@
 $EndComp
 $Comp
-L sonde~xilinx_schlib:74LS125 U2
+L sonde_xilinx_schlib:74LS125 U2
 U 2 1 3EBF7EDD
 P 1700 6900
@@
 	4650 2000 4650 1900
 $Comp
-L sonde~xilinx_schlib:74LS125 U1
+L sonde_xilinx_schlib:74LS125 U1
 U 3 1 3EBF7DB3
 P 5450 3300
@@
 $EndComp
 $Comp
-L sonde~xilinx_schlib:74LS125 U1
+L sonde_xilinx_schlib:74LS125 U1
 U 2 1 3EBF7DAD
 P 5450 2600
@@
 $EndComp
 $Comp
-L sonde~xilinx_schlib:74LS125 U1
+L sonde_xilinx_schlib:74LS125 U1
 U 1 1 3EBF7D9F
 P 5400 1900
@@
 $EndComp
 $Comp
-L sonde~xilinx_schlib:74LS125 U2
+L sonde_xilinx_schlib:74LS125 U2
 U 1 1 3EBF7D92
 P 4650 1600
@@
 	2200 1600 3700 1600
 $Comp
-L sonde~xilinx_schlib:R R9
+L sonde_xilinx_schlib:R R9
 U 1 1 3EBF7D33
 P 3950 4200
@@
 $EndComp
 $Comp
-L sonde~xilinx_schlib:R R10
+L sonde_xilinx_schlib:R R10
 U 1 1 3EBF7D31
 P 3950 3300
@@
 $EndComp
 $Comp
-L sonde~xilinx_schlib:R R8
+L sonde_xilinx_schlib:R R8
 U 1 1 4D528080
 P 3950 2900
@@
 $EndComp
 $Comp
-L sonde~xilinx_schlib:R R7
+L sonde_xilinx_schlib:R R7
 U 1 1 4D52807F
 P 3950 2600
@@
 $EndComp
 $Comp
-L sonde~xilinx_schlib:R R6
+L sonde_xilinx_schlib:R R6
 U 1 1 3EBF7D26
 P 3950 2250
@@
 $EndComp
 $Comp
-L sonde~xilinx_schlib:R R4
+L sonde_xilinx_schlib:R R4
 U 1 1 3EBF7D22
 P 3950 1600
@@
 $EndComp
 $Comp
-L sonde~xilinx_schlib:R R1
+L sonde_xilinx_schlib:R R1
 U 1 1 3EBF7D16
 P 3950 1000
@@
 $EndComp
 $Comp
-L sonde~xilinx_schlib:DB25 J1
+L sonde_xilinx_schlib:DB25 J1
 U 1 1 3EBF7D04
 P 1750 2800
@@
 Connection ~ 7650 1000
 $Comp
-L sonde~xilinx_schlib:GND #PWR017
+L sonde_xilinx_schlib:GND #PWR017
 U 1 1 5510FC05
 P 4950 2000

Commit message: Update demos
Parts:
- J1: footprint Connect:DB25M_CI -> Connector_Dsub:DSUB-25_Male_EdgeMount_P2.77mm
- J2: footprint Connect:DB9M_CI_INVERT -> Connector_Dsub:DSUB-9_Male_EdgeMount_P2.77mm
Changed lines of the file:
@@
 F 0 "J2" H 10700 4450 70  0000 C CNN
 F 1 "DB9MALE" H 10700 3353 70  0000 C CNN
-F 2 "Connect:DB9M_CI_INVERT" H 10700 3900 60  0001 C CNN
+F 2 "Connector_Dsub:DSUB-9_Male_EdgeMount_P2.77mm" H 10700 3900 60  0001 C CNN
 F 3 "" H 10700 3900 60  0001 C CNN
 	1    10700 3900
@@
 F 0 "J1" H 1800 4150 70  0000 C CNN
 F 1 "DB25MALE" H 1700 1450 70  0000 C CNN
-F 2 "Connect:DB25M_CI" H 1750 2800 60  0001 C CNN
+F 2 "Connector_Dsub:DSUB-25_Male_EdgeMount_P2.77mm" H 1750 2800 60  0001 C CNN
 F 3 "" H 1750 2800 60  0001 C CNN
 	1    1750 2800
