File: demos/flat_hierarchy/pic_sockets.sch (KiCad schematic (older format))
At the start: 8 parts, among them P2 SUPP28, P3 SUPP40, U1 24Cxx, U5 PIC_18_PINS, U6 PIC_8_PINS

Commit message: Update demos
Parts:
- C6, C7, C8: symbol C -> flat_hierarchy_schlib:C
- P2: symbol SUPP28 -> flat_hierarchy_schlib:SUPP28
- P3: symbol SUPP40 -> flat_hierarchy_schlib:SUPP40
- U1: symbol 24C16 -> flat_hierarchy_schlib:24C16
- U5: symbol PIC16F54 -> flat_hierarchy_schlib:PIC16F54
- U6: symbol PIC12C508A -> flat_hierarchy_schlib:PIC12C508A
Changed lines of the file:
@@
-EESchema Schematic File Version 2
-LIBS:flat_hierarchy_schlib
+EESchema Schematic File Version 4
 LIBS:flat_hierarchy-cache
-EELAYER 25 0
+EELAYER 26 0
 EELAYER END
 $Descr A4 11693 8268
@@
 	2200 6500 2200 6600
 $Comp
-L GND #PWR01
+L flat_hierarchy_schlib:GND #PWR01
 U 1 1 4639BE2E
 P 2200 7050
@@
 $EndComp
 $Comp
-L C C8
+L flat_hierarchy_schlib:C C8
 U 1 1 4639BE2C
 P 2200 6800
@@
 VCC_PIC
 $Comp
-L GND #PWR02
+L flat_hierarchy_schlib:GND #PWR02
 U 1 1 442A8794
 P 7700 5100
@@
 VCC_PIC
 $Comp
-L GND #PWR03
+L flat_hierarchy_schlib:GND #PWR03
 U 1 1 443CCA5D
 P 7700 4700
@@
 NoConn ~ 7700 2250
 $Comp
-L GND #PWR04
+L flat_hierarchy_schlib:GND #PWR04
 U 1 1 443697C7
 P 8900 3050
@@
 $EndComp
 $Comp
-L GND #PWR05
+L flat_hierarchy_schlib:GND #PWR05
 U 1 1 443697C3
 P 7700 2850
@@
 VPP-MCLR
 $Comp
-L SUPP28 P2
+L flat_hierarchy_schlib:SUPP28 P2
 U 1 1 4436967E
 P 8300 2800
@@
 $EndComp
 $Comp
-L GND #PWR06
+L flat_hierarchy_schlib:GND #PWR06
 U 1 1 442AA147
 P 1650 7050
@@
 $EndComp
 $Comp
-L C C7
+L flat_hierarchy_schlib:C C7
 U 1 1 442AA145
 P 1650 6800
@@
 $EndComp
 $Comp
-L GND #PWR07
+L flat_hierarchy_schlib:GND #PWR07
 U 1 1 442AA138
 P 2750 7050
@@
 $EndComp
 $Comp
-L VCC #PWR08
+L flat_hierarchy_schlib:VCC #PWR08
 U 1 1 442AA134
 P 2750 6600
@@
 $EndComp
 $Comp
-L C C6
+L flat_hierarchy_schlib:C C6
 U 1 1 442AA12B
 P 2750 6800
@@
 NoConn ~ 7700 4100
 $Comp
-L GND #PWR09
+L flat_hierarchy_schlib:GND #PWR09
 U 1 1 442A896A
 P 8900 4900
@@
 $EndComp
 $Comp
-L SUPP40 P3
+L flat_hierarchy_schlib:SUPP40 P3
 U 1 1 442A88ED
 P 8300 4950
@@
 NoConn ~ 3950 1300
 $Comp
-L GND #PWR010
+L flat_hierarchy_schlib:GND #PWR010
 U 1 1 442A8838
 P 2350 1450
@@
 CLOCK-RB6
 $Comp
-L 24C16 U1
+L flat_hierarchy_schlib:24C16 U1
 U 1 1 442A87F7
 P 3250 1400
@@
 NoConn ~ 2500 4250
 $Comp
-L PIC16F54 U5
+L flat_hierarchy_schlib:PIC16F54 U5
 U 1 1 442A81A7
 P 3300 4850
@@
 DATA-RB7
 $Comp
-L GND #PWR011
+L flat_hierarchy_schlib:GND #PWR011
 U 1 1 442A820F
 P 2300 4900
@@
 $EndComp
 $Comp
-L GND #PWR012
+L flat_hierarchy_schlib:GND #PWR012
 U 1 1 442A8205
 P 4000 2500
@@
 $EndComp
 $Comp
-L PIC12C508A U6
+L flat_hierarchy_schlib:PIC12C508A U6
 U 1 1 442A81A5
 P 3300 3000
@@
 $EndComp
 $Comp
-L VCC #PWR013
+L flat_hierarchy_schlib:VCC #PWR013
 U 1 1 53B84749
 P 3250 900
@@
 $EndComp
 $Comp
-L GND #PWR014
+L flat_hierarchy_schlib:GND #PWR014
 U 1 1 53B847AC
 P 3250 1900

Commit message: demos update
Parts:
- C6, C7, C8: footprint Discret:C1-1 -> discret:C1-1
- P2: footprint Sockets_DIP:DIP-28__300_ELL -> 28DIP-ELL300
- P3: footprint Sockets_DIP:DIP-40__600_ELL -> 40DIP-ELL600
- U1, U6: footprint Sockets_DIP:DIP-8__300_ELL -> dip_sockets:DIP-8__300_ELL
- U5: footprint Sockets_DIP:DIP-18__300_ELL -> dip_sockets:DIP-18__300_ELL
Changed lines of the file:
@@
 VPP-MCLR
 Wire Wire Line
-	1650 2500 1650 6600
-Wire Wire Line
-	1500 2500 2550 2500
+	1650 2500 1650 6200
+Wire Wire Line
+	1500 2500 1650 2500
 Wire Wire Line
 	8900 2250 9800 2250
@@
 Connection ~ 2350 1400
 Wire Wire Line
-	2350 1200 2350 1450
+	2350 1200 2350 1300
 Wire Wire Line
 	2350 1200 2550 1200
@@
 	2550 1400 2350 1400
 Wire Wire Line
-	3950 1600 10150 1600
-Wire Wire Line
-	3950 1500 10150 1500
+	3950 1600 4800 1600
+Wire Wire Line
+	3950 1500 4900 1500
 Wire Wire Line
 	9800 4100 8900 4100
@@
 	4000 2800 4800 2800
 Wire Wire Line
-	1500 3500 2550 3500
+	1500 3500 1750 3500
 Wire Wire Line
 	2300 4850 2300 4900
@@
 F 0 "C8" H 2250 6900 50  0000 L CNN
 F 1 "100nF" H 2250 6700 50  0000 L CNN
-F 2 "Discret:C1-1" H 2200 6800 60  0001 C CNN
+F 2 "discret:C1-1" H 2200 6800 60  0001 C CNN
 F 3 "" H 2200 6800 60  0001 C CNN
 	1    2200 6800
@@
 F 0 "P2" H 8300 3600 70  0000 C CNN
 F 1 "SUPP28" H 8300 1950 70  0000 C CNN
-F 2 "Sockets_DIP:DIP-28__300_ELL" H 8300 2800 60  0001 C CNN
+F 2 "28DIP-ELL300" H 8300 2800 60  0001 C CNN
 F 3 "" H 8300 2800 60  0001 C CNN
 	1    8300 2800
@@
 F 0 "C7" H 1700 6900 50  0000 L CNN
 F 1 "100nF" H 1700 6700 50  0000 L CNN
-F 2 "Discret:C1-1" H 1650 6800 60  0001 C CNN
+F 2 "discret:C1-1" H 1650 6800 60  0001 C CNN
 F 3 "" H 1650 6800 60  0001 C CNN
 	1    1650 6800
@@
 F 0 "C6" H 2800 6900 50  0000 L CNN
 F 1 "100nF" H 2800 6700 50  0000 L CNN
-F 2 "Discret:C1-1" H 2750 6800 60  0001 C CNN
+F 2 "discret:C1-1" H 2750 6800 60  0001 C CNN
 F 3 "" H 2750 6800 60  0001 C CNN
 	1    2750 6800
@@
 F 0 "P3" H 8300 6050 70  0000 C CNN
 F 1 "SUPP40" H 8300 3800 70  0000 C CNN
-F 2 "Sockets_DIP:DIP-40__600_ELL" H 8300 4950 60  0001 C CNN
+F 2 "40DIP-ELL600" H 8300 4950 60  0001 C CNN
 F 3 "" H 8300 4950 60  0001 C CNN
 	1    8300 4950
@@
 F 0 "U1" H 3400 1750 60  0000 C CNN
 F 1 "24Cxx" H 3450 1050 60  0000 C CNN
-F 2 "Sockets_DIP:DIP-8__300_ELL" H 3250 1400 60  0001 C CNN
+F 2 "dip_sockets:DIP-8__300_ELL" H 3250 1400 60  0001 C CNN
 F 3 "" H 3250 1400 60  0001 C CNN
 	1    3250 1400
@@
 F 0 "U5" H 3300 5600 60  0000 C CNN
 F 1 "PIC_18_PINS" H 3300 4050 60  0000 C CNN
-F 2 "Sockets_DIP:DIP-18__300_ELL" H 3300 4850 60  0001 C CNN
+F 2 "dip_sockets:DIP-18__300_ELL" H 3300 4850 60  0001 C CNN
 F 3 "" H 3300 4850 60  0001 C CNN
 	1    3300 4850
@@
 F 0 "U6" H 3250 3700 60  0000 C CNN
 F 1 "PIC_8_PINS" H 3300 2300 60  0000 C CNN
-F 2 "Sockets_DIP:DIP-8__300_ELL" H 3300 3000 60  0001 C CNN
+F 2 "dip_sockets:DIP-8__300_ELL" H 3300 3000 60  0001 C CNN
 F 3 "" H 3300 3000 60  0001 C CNN
 	1    3300 3000
@@
 $EndComp
 Wire Wire Line
-	4800 1600 4800 5000
-Connection ~ 4800 5000
+	4800 1600 4800 2800
 Connection ~ 4800 2800
 Wire Wire Line
 	4800 5000 4050 5000
 Wire Wire Line
-	4900 1500 4900 5150
+	4900 1500 4900 3200
 Connection ~ 4900 3200
 Wire Wire Line
-	9800 1500 9800 4100
+	9800 1500 9800 2250
 Connection ~ 4900 1500
 Connection ~ 9800 2250
 Wire Wire Line
-	9700 1600 9700 4000
+	9700 1600 9700 2150
 Connection ~ 4800 1600
 Connection ~ 9700 2150
 Wire Wire Line
-	9900 2950 9900 6200
+	9900 2950 9900 4800
 Wire Wire Line
 	5000 4850 5000 6200
 Wire Wire Line
-	9900 6200 1650 6200
+	9900 6200 6900 6200
 Connection ~ 9900 4800
 Wire Wire Line
-	1750 3500 1750 6100
+	1750 3500 1750 4700
 Connection ~ 5000 6200
 Connection ~ 1650 2500
@@
 	1750 6100 6700 6100
 Wire Wire Line
-	6700 6100 6700 2150
+	6700 6100 6700 4000
 Connection ~ 1750 4700
 Connection ~ 6700 4000
@@
 Wire Wire Line
 	1650 7000 1650 7050
+Wire Wire Line
+	2350 1300 2350 1400
+Wire Wire Line
+	2350 1400 2350 1450
+Wire Wire Line
+	4800 2800 4800 5000
+Wire Wire Line
+	4900 3200 4900 5150
+Wire Wire Line
+	4900 1500 9800 1500
+Wire Wire Line
+	9800 2250 9800 4100
+Wire Wire Line
+	4800 1600 9700 1600
+Wire Wire Line
+	9700 2150 9700 4000
+Wire Wire Line
+	9900 4800 9900 6200
+Wire Wire Line
+	5000 6200 1650 6200
+Wire Wire Line
+	1650 2500 2550 2500
+Wire Wire Line
+	1750 4700 1750 6100
+Wire Wire Line
+	6700 4000 6700 2150
+Wire Wire Line
+	6900 6200 5000 6200
+Wire Wire Line
+	1650 6200 1650 6500
+Wire Wire Line
+	1650 6500 1650 6600
+Wire Wire Line
+	9700 1600 10150 1600
+Wire Wire Line
+	9800 1500 10150 1500
+Wire Wire Line
+	1750 3500 2550 3500
 $EndSCHEMATC
