File: demos/kit-dev-coldfire-xilinx_5213/xilinx.sch (KiCad schematic (older format))
At the start: 21 parts, among them P1 CONN_6, P3 CONN_2X2, P4 CONN_20X2, U9 XCR3256-TQ144

Commit message: Update demo kit-dev-coldfire-xilinx_5213
Parts:
- C301: renamed from C51; symbol kit-dev-coldfire-xilinx_5213_schlib:C -> kit-coldfire_schlib:C
- C302: renamed from C52; symbol kit-dev-coldfire-xilinx_5213_schlib:C -> kit-coldfire_schlib:C
- C303: renamed from C53; symbol kit-dev-coldfire-xilinx_5213_schlib:C -> kit-coldfire_schlib:C
- C304: renamed from C54; symbol kit-dev-coldfire-xilinx_5213_schlib:C -> kit-coldfire_schlib:C
- C305: renamed from C55; symbol kit-dev-coldfire-xilinx_5213_schlib:C -> kit-coldfire_schlib:C
- C306: renamed from C56; symbol kit-dev-coldfire-xilinx_5213_schlib:C -> kit-coldfire_schlib:C
- C307: renamed from C57; symbol kit-dev-coldfire-xilinx_5213_schlib:C -> kit-coldfire_schlib:C
- C308: renamed from C58; symbol kit-dev-coldfire-xilinx_5213_schlib:C -> kit-coldfire_schlib:C
- C309: renamed from C59; symbol kit-dev-coldfire-xilinx_5213_schlib:C -> kit-coldfire_schlib:C
- C310: renamed from C60; symbol kit-dev-coldfire-xilinx_5213_schlib:C -> kit-coldfire_schlib:C
- C311: renamed from C61; symbol kit-dev-coldfire-xilinx_5213_schlib:C -> kit-coldfire_schlib:C
- D301: renamed from D8; symbol kit-dev-coldfire-xilinx_5213_schlib:LED -> kit-coldfire_schlib:LED
- D302: renamed from D9; symbol kit-dev-coldfire-xilinx_5213_schlib:LED -> kit-coldfire_schlib:LED
- P301: renamed from P1; symbol kit-dev-coldfire-xilinx_5213_schlib:CONN_6 -> kit-coldfire_schlib:CONN_6
- P302: renamed from P3; symbol kit-dev-coldfire-xilinx_5213_schlib:CONN_2X2 -> kit-coldfire_schlib:CONN_2X2
- P303: renamed from P4; symbol kit-dev-coldfire-xilinx_5213_schlib:CONN_20X2 -> kit-coldfire_schlib:CONN_20X2
- R301: renamed from R57; symbol kit-dev-coldfire-xilinx_5213_schlib:R -> kit-coldfire_schlib:R
- R302: renamed from R64; symbol kit-dev-coldfire-xilinx_5213_schlib:R -> kit-coldfire_schlib:R
- R303: renamed from R62; symbol kit-dev-coldfire-xilinx_5213_schlib:R -> kit-coldfire_schlib:R
- R304: renamed from R63; symbol kit-dev-coldfire-xilinx_5213_schlib:R -> kit-coldfire_schlib:R
- U301: renamed from U9; symbol kit-dev-coldfire-xilinx_5213_schlib:XCR3256-TQ144 -> kit-coldfire_schlib:XCR3256-TQ144

Commit message: Fixes in demo kit-dev-coldfire-xilinx_5213.
Parts:
- C301, C302, C303, C304, C305, C306, C307, C308, C309, C310, C311: footprint Resistor_SMD:R_0805_2012Metric -> Capacitor_SMD:C_0805_2012Metric
Changed lines of the file:
@@
 F 0 "C311" H 10650 6250 50  0000 L CNN
 F 1 "100nF" H 10600 6050 50  0000 L CNN
-F 2 "Resistor_SMD:R_0805_2012Metric" H 10600 6150 60  0001 C CNN
+F 2 "Capacitor_SMD:C_0805_2012Metric" H 10600 6150 60  0001 C CNN
 F 3 "" H 10600 6150 60  0001 C CNN
 	1    10600 6150
@@
 F 0 "C310" H 10350 6250 50  0000 L CNN
 F 1 "100nF" H 10300 6050 50  0000 L CNN
-F 2 "Resistor_SMD:R_0805_2012Metric" H 10300 6150 60  0001 C CNN
+F 2 "Capacitor_SMD:C_0805_2012Metric" H 10300 6150 60  0001 C CNN
 F 3 "" H 10300 6150 60  0001 C CNN
 	1    10300 6150
@@
 F 0 "C309" H 10050 6250 50  0000 L CNN
 F 1 "100nF" H 10000 6050 50  0000 L CNN
-F 2 "Resistor_SMD:R_0805_2012Metric" H 10000 6150 60  0001 C CNN
+F 2 "Capacitor_SMD:C_0805_2012Metric" H 10000 6150 60  0001 C CNN
 F 3 "" H 10000 6150 60  0001 C CNN
 	1    10000 6150
@@
 F 0 "C304" H 8550 6250 50  0000 L CNN
 F 1 "100nF" H 8500 6050 50  0000 L CNN
-F 2 "Resistor_SMD:R_0805_2012Metric" H 8500 6150 60  0001 C CNN
+F 2 "Capacitor_SMD:C_0805_2012Metric" H 8500 6150 60  0001 C CNN
 F 3 "" H 8500 6150 60  0001 C CNN
 	1    8500 6150
@@
 F 0 "C303" H 8250 6250 50  0000 L CNN
 F 1 "100nF" H 8200 6050 50  0000 L CNN
-F 2 "Resistor_SMD:R_0805_2012Metric" H 8200 6150 60  0001 C CNN
+F 2 "Capacitor_SMD:C_0805_2012Metric" H 8200 6150 60  0001 C CNN
 F 3 "" H 8200 6150 60  0001 C CNN
 	1    8200 6150
@@
 F 0 "C302" H 7950 6250 50  0000 L CNN
 F 1 "100nF" H 7900 6050 50  0000 L CNN
-F 2 "Resistor_SMD:R_0805_2012Metric" H 7900 6150 60  0001 C CNN
+F 2 "Capacitor_SMD:C_0805_2012Metric" H 7900 6150 60  0001 C CNN
 F 3 "" H 7900 6150 60  0001 C CNN
 	1    7900 6150
@@
 F 0 "C301" H 7650 6250 50  0000 L CNN
 F 1 "100nF" H 7600 6050 50  0000 L CNN
-F 2 "Resistor_SMD:R_0805_2012Metric" H 7600 6150 60  0001 C CNN
+F 2 "Capacitor_SMD:C_0805_2012Metric" H 7600 6150 60  0001 C CNN
 F 3 "" H 7600 6150 60  0001 C CNN
 	1    7600 6150
@@
 F 0 "C308" H 9750 6250 50  0000 L CNN
 F 1 "100nF" H 9700 6050 50  0000 L CNN
-F 2 "Resistor_SMD:R_0805_2012Metric" H 9700 6150 60  0001 C CNN
+F 2 "Capacitor_SMD:C_0805_2012Metric" H 9700 6150 60  0001 C CNN
 F 3 "" H 9700 6150 60  0001 C CNN
 	1    9700 6150
@@
 F 0 "C307" H 9450 6250 50  0000 L CNN
 F 1 "100nF" H 9400 6050 50  0000 L CNN
-F 2 "Resistor_SMD:R_0805_2012Metric" H 9400 6150 60  0001 C CNN
+F 2 "Capacitor_SMD:C_0805_2012Metric" H 9400 6150 60  0001 C CNN
 F 3 "" H 9400 6150 60  0001 C CNN
 	1    9400 6150
@@
 F 0 "C306" H 9150 6250 50  0000 L CNN
 F 1 "100nF" H 9100 6050 50  0000 L CNN
-F 2 "Resistor_SMD:R_0805_2012Metric" H 9100 6150 60  0001 C CNN
+F 2 "Capacitor_SMD:C_0805_2012Metric" H 9100 6150 60  0001 C CNN
 F 3 "" H 9100 6150 60  0001 C CNN
 	1    9100 6150
@@
 F 0 "C305" H 8850 6250 50  0000 L CNN
 F 1 "100nF" H 8800 6050 50  0000 L CNN
-F 2 "Resistor_SMD:R_0805_2012Metric" H 8800 6150 60  0001 C CNN
+F 2 "Capacitor_SMD:C_0805_2012Metric" H 8800 6150 60  0001 C CNN
 F 3 "" H 8800 6150 60  0001 C CNN
 	1    8800 6150
