File: demos/kit-dev-coldfire-xilinx_5213/kit-dev-coldfire-xilinx_5213.kicad_sch (KiCad schematic)
At the start: 66 parts, among them Q101 3906, U101 74AHC1G14, U102 MCF5213-LQFP100, Y101 8MHz

Commit message: Demo update
Parts:
- FB101, L101, L102: footprint Resistor_SMD:R_1206_3216Metric_Pad1.24x1.80mm_HandSolder -> Resistor_SMD:R_1206_3216Metric_Pad1.30x1.75mm_HandSolder
- LV101: footprint Package_TO_SOT_THT:TO-92_Molded_Narrow -> Package_TO_SOT_THT:TO-92

Commit message: Demo update
Parts:
- D101, D102: footprint Diode_SMD:D_SOT-23_ANK -> kit-dev-coldfire:D_SOT-23_ANK
