File: demos/video/pal-ntsc.kicad_sch (KiCad schematic)
At the start: 36 parts, among them U10 BT812, X2 30MHz

Commit message: Update demos.
Changed lines of the file:
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@@
-(kicad_sch (version 20210126) (generator eeschema)
+(kicad_sch (version 20210406) (generator eeschema)
   (paper "A3")
   (title_block
@@
     (stroke (width 0) (type solid) (color 0 0 0 0))
   )
-  (bus (pts (xy 270.51 78.74) (xy 270.51 81.28))
-    (stroke (width 0) (type solid) (color 0 0 0 0))
-  )
-  (bus (pts (xy 270.51 81.28) (xy 270.51 83.82))
-    (stroke (width 0) (type solid) (color 0 0 0 0))
-  )
-  (bus (pts (xy 270.51 83.82) (xy 270.51 86.36))
-    (stroke (width 0) (type solid) (color 0 0 0 0))
-  )
-  (bus (pts (xy 270.51 86.36) (xy 270.51 88.9))
-    (stroke (width 0) (type solid) (color 0 0 0 0))
-  )
-  (bus (pts (xy 270.51 88.9) (xy 270.51 91.44))
-    (stroke (width 0) (type solid) (color 0 0 0 0))
-  )
-  (bus (pts (xy 270.51 91.44) (xy 270.51 93.98))
-    (stroke (width 0) (type solid) (color 0 0 0 0))
-  )
-  (bus (pts (xy 270.51 93.98) (xy 270.51 96.52))
-    (stroke (width 0) (type solid) (color 0 0 0 0))
-  )
-  (bus (pts (xy 270.51 101.6) (xy 270.51 104.14))
-    (stroke (width 0) (type solid) (color 0 0 0 0))
-  )
-  (bus (pts (xy 270.51 104.14) (xy 270.51 106.68))
-    (stroke (width 0) (type solid) (color 0 0 0 0))
-  )
-  (bus (pts (xy 270.51 106.68) (xy 270.51 109.22))
-    (stroke (width 0) (type solid) (color 0 0 0 0))
-  )
-  (bus (pts (xy 270.51 109.22) (xy 270.51 111.76))
-    (stroke (width 0) (type solid) (color 0 0 0 0))
-  )
-  (bus (pts (xy 270.51 111.76) (xy 270.51 114.3))
-    (stroke (width 0) (type solid) (color 0 0 0 0))
-  )
-  (bus (pts (xy 270.51 114.3) (xy 270.51 116.84))
-    (stroke (width 0) (type solid) (color 0 0 0 0))
-  )
-  (bus (pts (xy 270.51 116.84) (xy 270.51 119.38))
-    (stroke (width 0) (type solid) (color 0 0 0 0))
-  )
-  (bus (pts (xy 270.51 124.46) (xy 270.51 127))
-    (stroke (width 0) (type solid) (color 0 0 0 0))
-  )
-  (bus (pts (xy 270.51 127) (xy 270.51 129.54))
-    (stroke (width 0) (type solid) (color 0 0 0 0))
-  )
-  (bus (pts (xy 270.51 129.54) (xy 270.51 132.08))
-    (stroke (width 0) (type solid) (color 0 0 0 0))
-  )
-  (bus (pts (xy 270.51 132.08) (xy 270.51 134.62))
-    (stroke (width 0) (type solid) (color 0 0 0 0))
-  )
-  (bus (pts (xy 270.51 134.62) (xy 270.51 137.16))
-    (stroke (width 0) (type solid) (color 0 0 0 0))
-  )
-  (bus (pts (xy 270.51 137.16) (xy 270.51 139.7))
-    (stroke (width 0) (type solid) (color 0 0 0 0))
-  )
-  (bus (pts (xy 270.51 139.7) (xy 270.51 142.24))
-    (stroke (width 0) (type solid) (color 0 0 0 0))
-  )
+  (bus (pts (xy 270.51 78.74) (xy 270.51 96.52))
+    (stroke (width 0) (type solid) (color 0 0 0 0))
+  )
+  (bus (pts (xy 270.51 101.6) (xy 270.51 119.38))
+    (stroke (width 0) (type solid) (color 0 0 0 0))
+  )
+  (bus (pts (xy 270.51 124.46) (xy 270.51 142.24))
+    (stroke (width 0) (type solid) (color 0 0 0 0))
+  )

Commit message: Demos update
Parts:
- U: renamed from C15; value 100nF -> (none); footprint Resistor_SMD:R_1206_3216Metric_Pad1.24x1.80mm_HandSolder -> (none)
- U: renamed from C16; value 100nF -> (none); footprint Resistor_SMD:R_1206_3216Metric_Pad1.24x1.80mm_HandSolder -> (none)
- U: renamed from X2; value 30MHz -> (none); footprint Crystal:Crystal_HC18-U_Vertical -> (none)
- U: renamed from C66; value 22pF -> (none); footprint Resistor_SMD:R_1206_3216Metric_Pad1.24x1.80mm_HandSolder -> (none)
- U: renamed from C11; value 100nF -> (none); footprint Resistor_SMD:R_1206_3216Metric_Pad1.24x1.80mm_HandSolder -> (none)
- U: renamed from C14; value 100nF -> (none); footprint Resistor_SMD:R_1206_3216Metric_Pad1.24x1.80mm_HandSolder -> (none)
- U: renamed from D2; value BAT46 -> (none); footprint Diode_THT:D_DO-34_SOD68_P7.62mm_Horizontal -> (none)
- U: renamed from R25; value 220K -> (none); footprint Resistor_SMD:R_1206_3216Metric_Pad1.24x1.80mm_HandSolder -> (none)
- U: renamed from L4; value 22uF -> (none); footprint Resistor_SMD:R_1812_4532Metric_Pad1.24x3.50mm_HandSolder -> (none)
- U: renamed from D1; value BAT46 -> (none); footprint Diode_THT:D_DO-34_SOD68_P7.62mm_Horizontal -> (none)
- U: renamed from R2; value 100 -> (none); footprint Resistor_SMD:R_1206_3216Metric_Pad1.24x1.80mm_HandSolder -> (none)
- U: renamed from C47; value 220pF -> (none); footprint Resistor_SMD:R_1206_3216Metric_Pad1.24x1.80mm_HandSolder -> (none)
- U: renamed from C4; value 100nF -> (none); footprint Resistor_SMD:R_1206_3216Metric_Pad1.24x1.80mm_HandSolder -> (none)
- U: renamed from C6; value 100nF -> (none); footprint Resistor_SMD:R_1206_3216Metric_Pad1.24x1.80mm_HandSolder -> (none)
- U: renamed from R35; value 470 -> (none); footprint Resistor_SMD:R_1206_3216Metric_Pad1.24x1.80mm_HandSolder -> (none)
- U: renamed from C3; value 100nF -> (none); footprint Resistor_SMD:R_1206_3216Metric_Pad1.24x1.80mm_HandSolder -> (none)
- U: renamed from C5; value 100nF -> (none); footprint Resistor_SMD:R_1206_3216Metric_Pad1.24x1.80mm_HandSolder -> (none)
- U: renamed from C62; value 47uF -> (none); footprint Resistor_SMD:R_1210_3225Metric_Pad1.24x2.70mm_HandSolder -> (none)
- U: renamed from C2; value 100nF -> (none); footprint Resistor_SMD:R_1206_3216Metric_Pad1.24x1.80mm_HandSolder -> (none)
- U: renamed from C10; value 100nF -> (none); footprint Resistor_SMD:R_1206_3216Metric_Pad1.24x1.80mm_HandSolder -> (none)
- U: renamed from C13; value 100nF -> (none); footprint Resistor_SMD:R_1206_3216Metric_Pad1.24x1.80mm_HandSolder -> (none)
- U: renamed from U10; value BT812 -> (none); footprint Package_QFP:PQFP-160_28x28mm_P0.65mm -> (none)
- U: renamed from R19; value 220 -> (none); footprint Resistor_SMD:R_1206_3216Metric_Pad1.24x1.80mm_HandSolder -> (none)
- U: renamed from R12; value 1K -> (none); footprint Resistor_SMD:R_1206_3216Metric_Pad1.24x1.80mm_HandSolder -> (none)
- U: renamed from C12; value 100nF -> (none); footprint Resistor_SMD:R_1206_3216Metric_Pad1.24x1.80mm_HandSolder -> (none)
- U: renamed from C1; value 100nF -> (none); footprint Resistor_SMD:R_1206_3216Metric_Pad1.24x1.80mm_HandSolder -> (none)
- U: renamed from D3; value BAT46 -> (none); footprint Diode_THT:D_DO-34_SOD68_P7.62mm_Horizontal -> (none)
- U: renamed from C7; value 100nF -> (none); footprint Resistor_SMD:R_1206_3216Metric_Pad1.24x1.80mm_HandSolder -> (none)
- U: renamed from D4; value BAT46 -> (none); footprint Diode_THT:D_DO-34_SOD68_P7.62mm_Horizontal -> (none)
- U: renamed from R20; value 220 -> (none); footprint Resistor_SMD:R_1206_3216Metric_Pad1.24x1.80mm_HandSolder -> (none)
- U: renamed from R27; value 27K -> (none); footprint Resistor_SMD:R_1206_3216Metric_Pad1.24x1.80mm_HandSolder -> (none)
- U: renamed from C9; value 100nF -> (none); footprint Resistor_SMD:R_1206_3216Metric_Pad1.24x1.80mm_HandSolder -> (none)
- U: renamed from R14; value 1M -> (none); footprint Resistor_SMD:R_1206_3216Metric_Pad1.24x1.80mm_HandSolder -> (none)
- U: renamed from C8; value 100nF -> (none); footprint Resistor_SMD:R_1206_3216Metric_Pad1.24x1.80mm_HandSolder -> (none)
- U: renamed from C65; value 22pF -> (none); footprint Resistor_SMD:R_1206_3216Metric_Pad1.24x1.80mm_HandSolder -> (none)
- U: renamed from R3; value 100 -> (none); footprint Resistor_SMD:R_1206_3216Metric_Pad1.24x1.80mm_HandSolder -> (none)
