File: demos/video/graphic.kicad_sch (KiCad schematic)
At the start: 34 parts

Commit message: Demos update.
Parts:
- C17, C18, C19, C20, C21, C22, C23, C70, C71, C72, C73: renamed from U; value (none) -> 100nF; footprint (none) -> Resistor_SMD:R_1206_3216Metric_Pad1.24x1.80mm_HandSolder
- C49, C50: renamed from U; value (none) -> 22pF; footprint (none) -> Capacitor_THT:C_Disc_D3.0mm_W2.0mm_P2.50mm
- C56, C57: renamed from U; value (none) -> 4.7uF; footprint (none) -> Capacitor_Tantalum_SMD:CP_EIA-3528-21_Kemet-B_Pad1.63x2.40mm_HandSolder
- C63: renamed from U; value (none) -> 47uF; footprint (none) -> Resistor_SMD:R_1210_3225Metric_Pad1.24x2.70mm_HandSolder
- D6: renamed from U; value (none) -> LED; footprint (none) -> Discret:LEDV
- P10, P11, P12, P9: renamed from U; value (none) -> CONN_1; footprint (none) -> Connector_PinHeader_2.54mm:PinHeader_1x01_P2.54mm_Vertical
- P4: renamed from U; value (none) -> CONN_2; footprint (none) -> Connector_PinHeader_2.54mm:PinHeader_1x02_P2.54mm_Vertical
- P5: renamed from U; value (none) -> CONN_5; footprint (none) -> Connector_PinHeader_2.54mm:PinHeader_1x05_P2.54mm_Vertical
- R1: renamed from U; value (none) -> 10; footprint (none) -> Resistor_SMD:R_1206_3216Metric_Pad1.24x1.80mm_HandSolder
- R13: renamed from U; value (none) -> 1K; footprint (none) -> Resistor_SMD:R_1206_3216Metric_Pad1.24x1.80mm_HandSolder
- R21: renamed from U; value (none) -> 220; footprint (none) -> Resistor_SMD:R_1206_3216Metric_Pad1.24x1.80mm_HandSolder
- R26: renamed from U; value (none) -> 220K; footprint (none) -> Resistor_SMD:R_1206_3216Metric_Pad1.24x1.80mm_HandSolder
- R48: renamed from U; value (none) -> 10K; footprint (none) -> Resistor_SMD:R_1206_3216Metric_Pad1.24x1.80mm_HandSolder
- U2: renamed from U; value (none) -> 4C4001; footprint (none) -> Package_SO:SOIC-28W_7.5x17.9mm_P1.27mm
- U21: renamed from U; value (none) -> XC1736APD8; footprint (none) -> Package_DIP:DIP-8_W7.62mm
- U23: renamed from U; value (none) -> XC4003/PQ100; footprint (none) -> Package_QFP:PQFP-100_14x20mm_P0.65mm
- U24: renamed from U; value (none) -> XC4005-PQ160; footprint (none) -> Package_QFP:PQFP-160_28x28mm_P0.65mm
- U7: renamed from U; value (none) -> AV9173; footprint (none) -> Package_SO:SSOP-8_3.95x5.21x3.27mm_P1.27mm
- X1: renamed from U; value (none) -> 10MHz; footprint (none) -> Crystal:Crystal_HC18-U_Vertical

Commit message: Demo update
Other:
- moved on the sheet: R48
