File: demos/video/rams.kicad_sch (KiCad schematic)
At the start: 8 parts

Commit message: Demos update.
Parts:
- U12, U13, U14, U15, U16, U17, U18, U19: renamed from U; value (none) -> SIM4X32; footprint (none) -> footprints:sim72
Changed lines of the file:
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@@
-(kicad_sch (version 20220822) (generator eeschema)
+(kicad_sch (version 20221004) (generator eeschema)
   (paper "A3")
   (title_block
@@
   )
   (symbol (lib_id "video_schlib:SIM4X32") (at 307.34 189.23 0) (unit 1)
-    (in_bom yes) (on_board yes)
-    (default_instance (reference "U") (unit 1) (value "") (footprint ""))
-    (property "Reference" "U" (id 0) (at 307.34 175.26 0)
+    (in_bom yes) (on_board yes) (dnp no)
+    (property "Reference" "U13" (at 307.34 175.26 0)
       (effects (font (size 1.778 1.778)))
     )
-    (property "Value" "" (id 1) (at 318.77 240.03 0)
+    (property "Value" "SIM4X32" (at 318.77 240.03 0)
       (effects (font (size 1.778 1.778)))
     )
-    (property "Footprint" "" (id 2) (at 307.34 189.23 0)
+    (property "Footprint" "footprints:sim72" (at 307.34 189.23 0)
       (effects (font (size 1.524 1.524)) hide)
     )
-    (property "Datasheet" "" (id 3) (at 307.34 189.23 0)
+    (property "Datasheet" "" (at 307.34 189.23 0)
       (effects (font (size 1.524 1.524)) hide)
     )
@@
     (pin "8")
     (pin "9")
+    (instances
+      (project "video"
+        (path "/f54f2c44-70ae-46db-88a1-bf696c289e90/00000000-0000-0000-0000-00004bf03685"
+          (reference "U13") (unit 1) (value "SIM4X32") (footprint "footprints:sim72")
+        )
+      )
+    )
   )
   (symbol (lib_id "video_schlib:SIM4X32") (at 163.83 189.23 0) (unit 1)
-    (in_bom yes) (on_board yes)
-    (default_instance (reference "U") (unit 1) (value "") (footprint ""))
-    (property "Reference" "U" (id 0) (at 163.83 175.26 0)
+    (in_bom yes) (on_board yes) (dnp no)
+    (property "Reference" "U12" (at 163.83 175.26 0)
       (effects (font (size 1.778 1.778)))
     )
-    (property "Value" "" (id 1) (at 175.26 240.03 0)
+    (property "Value" "SIM4X32" (at 175.26 240.03 0)
       (effects (font (size 1.778 1.778)))
     )
-    (property "Footprint" "" (id 2) (at 163.83 189.23 0)
+    (property "Footprint" "footprints:sim72" (at 163.83 189.23 0)
       (effects (font (size 1.524 1.524)) hide)
     )
-    (property "Datasheet" "" (id 3) (at 163.83 189.23 0)
+    (property "Datasheet" "" (at 163.83 189.23 0)
       (effects (font (size 1.524 1.524)) hide)
     )
@@
     (pin "8")
     (pin "9")
+    (instances
+      (project "video"
+        (path "/f54f2c44-70ae-46db-88a1-bf696c289e90/00000000-0000-0000-0000-00004bf03685"
+          (reference "U12") (unit 1) (value "SIM4X32") (footprint "footprints:sim72")
+        )
+      )
+    )
   )
   (symbol (lib_id "video_schlib:SIM4X32") (at 236.22 189.23 0) (unit 1)
-    (in_bom yes) (on_board yes)
-    (default_instance (reference "U") (unit 1) (value "") (footprint ""))
-    (property "Reference" "U" (id 0) (at 236.22 175.26 0)
+    (in_bom yes) (on_board yes) (dnp no)
+    (property "Reference" "U14" (at 236.22 175.26 0)
       (effects (font (size 1.778 1.778)))
     )
-    (property "Value" "" (id 1) (at 247.65 240.03 0)
+    (property "Value" "SIM4X32" (at 247.65 240.03 0)
       (effects (font (size 1.778 1.778)))
     )
-    (property "Footprint" "" (id 2) (at 236.22 189.23 0)
+    (property "Footprint" "footprints:sim72" (at 236.22 189.23 0)
       (effects (font (size 1.524 1.524)) hide)
     )
-    (property "Datasheet" "" (id 3) (at 236.22 189.23 0)
+    (property "Datasheet" "" (at 236.22 189.23 0)
       (effects (font (size 1.524 1.524)) hide)
     )
@@
     (pin "8")
     (pin "9")
+    (instances
+      (project "video"
+        (path "/f54f2c44-70ae-46db-88a1-bf696c289e90/00000000-0000-0000-0000-00004bf03685"
+          (reference "U14") (unit 1) (value "SIM4X32") (footprint "footprints:sim72")
+        )
+      )
+    )
   )
   (symbol (lib_id "video_schlib:SIM4X32") (at 91.44 189.23 0) (unit 1)
-    (in_bom yes) (on_board yes)
-    (default_instance (reference "U") (unit 1) (value "") (footprint ""))
-    (property "Reference" "U" (id 0) (at 91.44 175.26 0)
+    (in_bom yes) (on_board yes) (dnp no)
+    (property "Reference" "U16" (at 91.44 175.26 0)
       (effects (font (size 1.778 1.778)))
     )
-    (property "Value" "" (id 1) (at 102.87 240.03 0)
+    (property "Value" "SIM4X32" (at 102.87 240.03 0)
       (effects (font (size 1.778 1.778)))
     )
-    (property "Footprint" "" (id 2) (at 91.44 189.23 0)
+    (property "Footprint" "footprints:sim72" (at 91.44 189.23 0)
       (effects (font (size 1.524 1.524)) hide)
     )
-    (property "Datasheet" "" (id 3) (at 91.44 189.23 0)
+    (property "Datasheet" "" (at 91.44 189.23 0)
       (effects (font (size 1.524 1.524)) hide)
     )
@@
     (pin "8")
     (pin "9")
+    (instances
+      (project "video"
+        (path "/f54f2c44-70ae-46db-88a1-bf696c289e90/00000000-0000-0000-0000-00004bf03685"
+          (reference "U16") (unit 1) (value "SIM4X32") (footprint "footprints:sim72")
+        )
+      )
+    )
   )
   (symbol (lib_id "video_schlib:SIM4X32") (at 307.34 76.2 0) (unit 1)
-    (in_bom yes) (on_board yes)
-    (default_instance (reference "U") (unit 1) (value "") (footprint ""))
-    (property "Reference" "U" (id 0) (at 307.34 62.23 0)
+    (in_bom yes) (on_board yes) (dnp no)
+    (property "Reference" "U15" (at 307.34 62.23 0)
       (effects (font (size 1.778 1.778)))
     )
-    (property "Value" "" (id 1) (at 318.77 127 0)
+    (property "Value" "SIM4X32" (at 318.77 127 0)
       (effects (font (size 1.778 1.778)))
     )
-    (property "Footprint" "" (id 2) (at 307.34 76.2 0)
+    (property "Footprint" "footprints:sim72" (at 307.34 76.2 0)
       (effects (font (size 1.524 1.524)) hide)
     )
-    (property "Datasheet" "" (id 3) (at 307.34 76.2 0)
+    (property "Datasheet" "" (at 307.34 76.2 0)
       (effects (font (size 1.524 1.524)) hide)
     )
@@
     (pin "8")
     (pin "9")
+    (instances
+      (project "video"
+        (path "/f54f2c44-70ae-46db-88a1-bf696c289e90/00000000-0000-0000-0000-00004bf03685"
+          (reference "U15") (unit 1) (value "SIM4X32") (footprint "footprints:sim72")
+        )
+      )
+    )
   )
   (symbol (lib_id "video_schlib:SIM4X32") (at 236.22 76.2 0) (unit 1)
-    (in_bom yes) (on_board yes)
-    (default_instance (reference "U") (unit 1) (value "") (footprint ""))
-    (property "Reference" "U" (id 0) (at 236.22 62.23 0)
+    (in_bom yes) (on_board yes) (dnp no)
+    (property "Reference" "U17" (at 236.22 62.23 0)
       (effects (font (size 1.778 1.778)))
     )
-    (property "Value" "" (id 1) (at 247.65 127 0)
+    (property "Value" "SIM4X32" (at 247.65 127 0)
       (effects (font (size 1.778 1.778)))
     )
-    (property "Footprint" "" (id 2) (at 236.22 76.2 0)
+    (property "Footprint" "footprints:sim72" (at 236.22 76.2 0)
       (effects (font (size 1.524 1.524)) hide)
     )
-    (property "Datasheet" "" (id 3) (at 236.22 76.2 0)
+    (property "Datasheet" "" (at 236.22 76.2 0)
       (effects (font (size 1.524 1.524)) hide)
     )
@@
     (pin "8")
     (pin "9")
+    (instances
+      (project "video"
+        (path "/f54f2c44-70ae-46db-88a1-bf696c289e90/00000000-0000-0000-0000-00004bf03685"
+          (reference "U17") (unit 1) (value "SIM4X32") (footprint "footprints:sim72")
+        )
+      )
+    )
   )
   (symbol (lib_id "video_schlib:SIM4X32") (at 163.83 76.2 0) (unit 1)
-    (in_bom yes) (on_board yes)
-    (default_instance (reference "U") (unit 1) (value "") (footprint ""))
-    (property "Reference" "U" (id 0) (at 163.83 62.23 0)
+    (in_bom yes) (on_board yes) (dnp no)
+    (property "Reference" "U18" (at 163.83 62.23 0)
       (effects (font (size 1.778 1.778)))
     )
-    (property "Value" "" (id 1) (at 175.26 127 0)
+    (property "Value" "SIM4X32" (at 175.26 127 0)
       (effects (font (size 1.778 1.778)))
     )
-    (property "Footprint" "" (id 2) (at 163.83 76.2 0)
+    (property "Footprint" "footprints:sim72" (at 163.83 76.2 0)
       (effects (font (size 1.524 1.524)) hide)
     )
-    (property "Datasheet" "" (id 3) (at 163.83 76.2 0)
+    (property "Datasheet" "" (at 163.83 76.2 0)
       (effects (font (size 1.524 1.524)) hide)
     )
@@
     (pin "8")
     (pin "9")
+    (instances
+      (project "video"
+        (path "/f54f2c44-70ae-46db-88a1-bf696c289e90/00000000-0000-0000-0000-00004bf03685"
+          (reference "U18") (unit 1) (value "SIM4X32") (footprint "footprints:sim72")
+        )
+      )
+    )
   )
   (symbol (lib_id "video_schlib:SIM4X32") (at 91.44 76.2 0) (unit 1)
-    (in_bom yes) (on_board yes)
-    (default_instance (reference "U") (unit 1) (value "") (footprint ""))
-    (property "Reference" "U" (id 0) (at 91.44 62.23 0)
+    (in_bom yes) (on_board yes) (dnp no)
+    (property "Reference" "U19" (at 91.44 62.23 0)
       (effects (font (size 1.778 1.778)))
     )
-    (property "Value" "" (id 1) (at 102.87 127 0)
+    (property "Value" "SIM4X32" (at 102.87 127 0)
       (effects (font (size 1.778 1.778)))
     )
-    (property "Footprint" "" (id 2) (at 91.44 76.2 0)
+    (property "Footprint" "footprints:sim72" (at 91.44 76.2 0)
       (effects (font (size 1.524 1.524)) hide)
     )
-    (property "Datasheet" "" (id 3) (at 91.44 76.2 0)
+    (property "Datasheet" "" (at 91.44 76.2 0)
       (effects (font (size 1.524 1.524)) hide)
     )
@@
     (pin "8")
     (pin "9")
+    (instances
+      (project "video"
+        (path "/f54f2c44-70ae-46db-88a1-bf696c289e90/00000000-0000-0000-0000-00004bf03685"
+          (reference "U19") (unit 1) (value "SIM4X32") (footprint "footprints:sim72")
+        )
+      )
+    )
   )
 )
