File: qa/eeschema/data/netlists/video/graphic.kicad_sch (KiCad schematic)
At the start: 34 parts, among them P10 CONN_1, P11 CONN_1, P12 CONN_1, P4 CONN_2, P5 CONN_5, P9 CONN_1, U2 4C4001, U21 XC1736APD8, U23 XC4003/PQ100, U24 XC4005-PQ160, U7 AV9173, X1 10MHz

Commit message: Update netlist QA testcases to new file format
Parts:
- removed C17, C18, C19, C20: 100nF, Resistor_SMD:R_1206_3216Metric_Pad1.24x1.80mm_HandSolder, symbol video_schlib:C
- removed C49, C50: 22pF, Capacitor_THT:C_Disc_D3.0mm_W2.0mm_P2.50mm, symbol video_schlib:C
- removed C56, C57: 4.7uF, Capacitor_Tantalum_SMD:CP_EIA-3528-21_Kemet-B_Pad1.63x2.40mm_HandSolder, symbol video_schlib:CP
- removed R26: 220K, Resistor_SMD:R_1206_3216Metric_Pad1.24x1.80mm_HandSolder, symbol video_schlib:R
Connections:
- net GND: now also X1.2
- net VCC: now also X1.1
- net XTAL_I: now also X1.1
- net at R21.1, X1.1: now also X1.2
Changed lines of the file:
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@@
-(kicad_sch (version 20200310) (host eeschema "(5.99.0-1545-g9916f24fa)")
-  (page "A3")
+(kicad_sch (version 20200512) (host eeschema "(5.99.0-1712-g5a9e69b14)")
+  (page 7 8)
+  (paper "A3")
   (title_block
     (title "Video")
@@
     (comment 1 "Xilinxs")
   )
+  (junction (at 22.86 45.72))
+  (junction (at 59.69 224.79))
+  (junction (at 68.58 185.42))
+  (junction (at 69.85 259.08))
+  (junction (at 69.85 271.78))
+  (junction (at 73.66 55.88))
+  (junction (at 76.2 35.56))
+  (junction (at 76.2 185.42))
+  (junction (at 78.74 259.08))
+  (junction (at 78.74 271.78))
+  (junction (at 81.28 45.72))
+  (junction (at 87.63 31.75))
+  (junction (at 87.63 38.1))
+  (junction (at 87.63 40.64))
+  (junction (at 88.9 259.08))
+  (junction (at 88.9 271.78))
+  (junction (at 97.79 259.08))
+  (junction (at 97.79 271.78))
+  (junction (at 106.68 259.08))
+  (junction (at 106.68 271.78))
+  (junction (at 115.57 259.08))
+  (junction (at 115.57 271.78))
+  (junction (at 129.54 259.08))
+  (junction (at 129.54 271.78))
+  (junction (at 138.43 259.08))
+  (junction (at 138.43 271.78))
+  (junction (at 147.32 259.08))
   (junction (at 147.32 271.78))
+  (junction (at 185.42 134.62))
+  (junction (at 187.96 134.62))
+  (junction (at 208.28 134.62))
+  (junction (at 208.28 139.7))
+  (junction (at 299.72 73.66))
   (junction (at 299.72 76.2))
-  (junction (at 68.58 185.42))
-  (junction (at 299.72 73.66))
-  (junction (at 138.43 271.78))
-  (junction (at 129.54 259.08))
-  (junction (at 78.74 271.78))
-  (junction (at 76.2 35.56))
-  (junction (at 106.68 259.08))
-  (junction (at 115.57 259.08))
-  (junction (at 88.9 259.08))
-  (junction (at 208.28 139.7))
-  (junction (at 88.9 271.78))
-  (junction (at 76.2 185.42))
-  (junction (at 87.63 31.75))
-  (junction (at 106.68 271.78))
-  (junction (at 69.85 259.08))
-  (junction (at 97.79 259.08))
-  (junction (at 69.85 271.78))
-  (junction (at 81.28 45.72))
-  (junction (at 185.42 134.62))
-  (junction (at 138.43 259.08))
-  (junction (at 87.63 40.64))
-  (junction (at 115.57 271.78))
-  (junction (at 187.96 134.62))
-  (junction (at 78.74 259.08))
-  (junction (at 129.54 271.78))
-  (junction (at 147.32 259.08))
-  (junction (at 59.69 224.79))
-  (junction (at 97.79 271.78))
-  (junction (at 87.63 38.1))
-  (junction (at 208.28 134.62))
-  (junction (at 22.86 45.72))
-  (junction (at 73.66 55.88))
+  (no_connect (at 63.5 43.18))
+  (no_connect (at 87.63 53.34))
+  (no_connect (at 140.97 109.22))
+  (no_connect (at 140.97 91.44))
   (no_connect (at 140.97 124.46))
+  (no_connect (at 358.14 144.78))
+  (no_connect (at 140.97 43.18))
+  (no_connect (at 140.97 38.1))
+  (no_connect (at 87.63 60.96))
   (no_connect (at 140.97 129.54))
+  (no_connect (at 110.49 219.71))
+  (no_connect (at 358.14 208.28))
   (no_connect (at 140.97 119.38))
+  (no_connect (at 87.63 63.5))
+  (no_connect (at 140.97 45.72))
+  (no_connect (at 140.97 147.32))
+  (no_connect (at 140.97 48.26))
   (no_connect (at 140.97 144.78))
-  (no_connect (at 87.63 63.5))
-  (no_connect (at 140.97 48.26))
-  (no_connect (at 358.14 144.78))
-  (no_connect (at 140.97 147.32))
-  (no_connect (at 63.5 43.18))
-  (no_connect (at 140.97 38.1))
-  (no_connect (at 358.14 208.28))
-  (no_connect (at 87.63 53.34))
-  (no_connect (at 110.49 219.71))
-  (no_connect (at 140.97 109.22))
-  (no_connect (at 140.97 43.18))
-  (no_connect (at 87.63 60.96))
-  (no_connect (at 140.97 91.44))
-  (no_connect (at 140.97 45.72))
   (wire (pts (xy 20.32 35.56) (xy 20.32 55.88)))
   (wire (pts (xy 20.32 55.88) (xy 73.66 55.88)))

Commit message: Convert video QA project to new format
Parts:
- added C17, C18, C19, C20: 100nF, Resistor_SMD:R_1206_3216Metric_Pad1.24x1.80mm_HandSolder, symbol video_schlib:C
- added C49, C50: 22pF, Capacitor_THT:C_Disc_D3.0mm_W2.0mm_P2.50mm, symbol video_schlib:C
- added C56, C57: 4.7uF, Capacitor_Tantalum_SMD:CP_EIA-3528-21_Kemet-B_Pad1.63x2.40mm_HandSolder, symbol video_schlib:CP
- added R26: 220K, Resistor_SMD:R_1206_3216Metric_Pad1.24x1.80mm_HandSolder, symbol video_schlib:R
Connections:
- net GND: now also C17.2, C18.2, C19.2, C20.2, C49.2, C50.2, C56.2, C57.2; no longer X1.2
- net VCC: now also C17.1, C18.1, C19.1, C20.1, C56.1, C57.1; no longer X1.1
- net XTAL_I: now also C50.1, R26.1; no longer X1.1
- net at P4.1 (P1), R48.2, U23.29 (M2): no longer U23.25 (M1), U23.27 (M0)
- net at R21.1, X1.1: now also C49.1, R26.2; no longer X1.2
Changed lines of the file:
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@@
-(kicad_sch (version 20200512) (host eeschema "(5.99.0-1712-g5a9e69b14)")
-  (page 7 8)
+(kicad_sch (version 20200512) (host eeschema "(5.99.0-1722-g89c46e683-dirty)")
+  (page 1 8)
   (paper "A3")
   (title_block
@@
   (junction (at 81.28 45.72))
   (junction (at 87.63 31.75))
-  (junction (at 87.63 38.1))
-  (junction (at 87.63 40.64))
   (junction (at 88.9 259.08))
   (junction (at 88.9 271.78))
@@
   (junction (at 299.72 73.66))
   (junction (at 299.72 76.2))
+  (no_connect (at 140.97 48.26))
+  (no_connect (at 140.97 119.38))
+  (no_connect (at 140.97 124.46))
+  (no_connect (at 87.63 60.96))
+  (no_connect (at 140.97 144.78))
   (no_connect (at 63.5 43.18))
+  (no_connect (at 140.97 147.32))
+  (no_connect (at 140.97 43.18))
   (no_connect (at 87.63 53.34))
+  (no_connect (at 358.14 144.78))
+  (no_connect (at 140.97 91.44))
+  (no_connect (at 140.97 129.54))
+  (no_connect (at 140.97 38.1))
+  (no_connect (at 140.97 45.72))
   (no_connect (at 140.97 109.22))
-  (no_connect (at 140.97 91.44))
-  (no_connect (at 140.97 124.46))
-  (no_connect (at 358.14 144.78))
-  (no_connect (at 140.97 43.18))
-  (no_connect (at 140.97 38.1))
-  (no_connect (at 87.63 60.96))
-  (no_connect (at 140.97 129.54))
   (no_connect (at 110.49 219.71))
+  (no_connect (at 87.63 63.5))
   (no_connect (at 358.14 208.28))
-  (no_connect (at 140.97 119.38))
-  (no_connect (at 87.63 63.5))
-  (no_connect (at 140.97 45.72))
-  (no_connect (at 140.97 147.32))
-  (no_connect (at 140.97 48.26))
-  (no_connect (at 140.97 144.78))
   (wire (pts (xy 20.32 35.56) (xy 20.32 55.88)))
   (wire (pts (xy 20.32 55.88) (xy 73.66 55.88)))
@@
   (wire (pts (xy 85.09 229.87) (xy 85.09 231.14)))
   (wire (pts (xy 87.63 27.94) (xy 87.63 31.75)))
-  (wire (pts (xy 87.63 31.75) (xy 87.63 38.1)))
-  (wire (pts (xy 87.63 38.1) (xy 87.63 40.64)))
-  (wire (pts (xy 87.63 40.64) (xy 87.63 43.18)))
+  (wire (pts (xy 87.63 31.75) (xy 87.63 43.18)))
   (wire (pts (xy 87.63 99.06) (xy 74.93 99.06)))
   (wire (pts (xy 87.63 101.6) (xy 74.93 101.6)))
