File: qa/data/issue2528.kicad_pcb (KiCad board)
At the start: 2 copper layers, 30 x 25 mm, 6 parts, among them Q1 Q_NPN_Darlington_ECBC

Commit message: Fix false test failures.
Changed lines of the file:
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@@
   (segment (start 162.8425 107) (end 165.5575 107) (width 0.25) (layer "F.Cu") (net 2))
   (segment (start 165.5575 107) (end 165.5575 110.8) (width 0.25) (layer "F.Cu") (net 2))
-  (segment (start 167.6425 109.3075) (end 167.65 109.3) (width 0.25) (layer "F.Cu") (net 3))
   (segment (start 157.2 98.4425) (end 157.2 99.5) (width 0.25) (layer "F.Cu") (net 3))
   (segment (start 157.2 99.5) (end 157.2 100.5575) (width 0.25) (layer "F.Cu") (net 3))
@@
   (segment (start 160.875001 102.725001) (end 160.875001 106.882499) (width 0.25) (layer "F.Cu") (net 5))
   (segment (start 157.2 102.6425) (end 160.7925 102.6425) (width 0.25) (layer "F.Cu") (net 5))
-  (segment (start 160.7925 102.6425) (end 160.875001 102.725001) (width 0.25) (layer "F.Cu") (net 5))
-  (segment (start 160.875001 106.882499) (end 160.7575 107) (width 0.25) (layer "F.Cu") (net 5))
   (zone (net 4) (net_name "/Col") (layer "F.Cu") (hatch edge 0.508)
     (priority 2)
