File: demos/simulation/subsheets/subsheet1.kicad_sch (KiCad schematic)
At the start: 3 parts

Commit message: Update some demos
Parts:
- U: renamed from C2; value 1u -> (none)
- U: renamed from R6; value 100 -> (none)
- U: renamed from R4; value 100 -> (none)
Changed lines of the file:
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@@
-(kicad_sch (version 20220104) (generator eeschema)
+(kicad_sch (version 20220404) (generator eeschema)
   (paper "A4")
   (junction (at 161.29 87.63) (diameter 0) (color 0 0 0 0)
@@
     (effects (font (size 1.27 1.27)) (justify right))
   )
-  (hierarchical_label "out" (shape input) (at 173.99 87.63 0) (fields_autoplaced)
+  (hierarchical_label "out" (shape output) (at 173.99 87.63 0) (fields_autoplaced)
     (effects (font (size 1.27 1.27)) (justify left))
   )
   (symbol (lib_id "Device:C") (at 161.29 95.25 0) (unit 1)
-    (in_bom yes) (on_board yes)
-    (property "Reference" "C2" (id 0) (at 165.1 94.615 0)
+    (in_bom yes) (on_board yes) (fields_autoplaced)
+    (default_instance (reference "U") (unit 1) (value "") (footprint ""))
+    (property "Reference" "U" (id 0) (at 164.211 94.6555 0)
       (effects (font (size 1.27 1.27)) (justify left))
     )
-    (property "Value" "1u" (id 1) (at 165.1 96.52 0)
+    (property "Value" "" (id 1) (at 164.211 96.4177 0)
       (effects (font (size 1.27 1.27)) (justify left))
     )
@@
   (symbol (lib_id "power:GND") (at 161.29 99.695 0) (unit 1)
     (in_bom yes) (on_board yes) (fields_autoplaced)
-    (property "Reference" "#PWR05" (id 0) (at 161.29 106.045 0)
+    (default_instance (reference "U") (unit 1) (value "") (footprint ""))
+    (property "Reference" "U" (id 0) (at 161.29 106.045 0)
       (effects (font (size 1.27 1.27)) hide)
     )
-    (property "Value" "GND" (id 1) (at 161.29 103.505 0)
+    (property "Value" "" (id 1) (at 161.29 103.505 0)
       (effects (font (size 1.27 1.27)))
     )
@@
   )
   (symbol (lib_id "Device:R") (at 168.91 87.63 90) (unit 1)
-    (in_bom yes) (on_board yes)
-    (property "Reference" "R6" (id 0) (at 168.275 85.09 0)
-      (effects (font (size 1.27 1.27)) (justify left))
+    (in_bom yes) (on_board yes) (fields_autoplaced)
+    (default_instance (reference "U") (unit 1) (value "") (footprint ""))
+    (property "Reference" "U" (id 0) (at 168.91 83.7819 90)
+      (effects (font (size 1.27 1.27)))
     )
-    (property "Value" "100" (id 1) (at 170.18 85.09 0)
-      (effects (font (size 1.27 1.27)) (justify left))
+    (property "Value" "" (id 1) (at 168.91 85.5441 90)
+      (effects (font (size 1.27 1.27)))
     )
     (property "Footprint" "" (id 2) (at 168.91 89.408 90)
@@
   )
   (symbol (lib_id "Device:R") (at 153.67 87.63 90) (unit 1)
-    (in_bom yes) (on_board yes)
-    (property "Reference" "R4" (id 0) (at 153.035 85.09 0)
-      (effects (font (size 1.27 1.27)) (justify left))
+    (in_bom yes) (on_board yes) (fields_autoplaced)
+    (default_instance (reference "U") (unit 1) (value "") (footprint ""))
+    (property "Reference" "U" (id 0) (at 153.67 83.7819 90)
+      (effects (font (size 1.27 1.27)))
     )
-    (property "Value" "100" (id 1) (at 154.94 85.09 0)
-      (effects (font (size 1.27 1.27)) (justify left))
+    (property "Value" "" (id 1) (at 153.67 85.5441 90)
+      (effects (font (size 1.27 1.27)))
     )
     (property "Footprint" "" (id 2) (at 153.67 89.408 90)
