File: demos/complex_hierarchy/complex_hierarchy.kicad_pcb (KiCad board)
At the start: 2 copper layers, 100.3 x 80 mm, 68 parts, among them P1 CONN_2, P2 CONN_2, P3 CONN_2, P4 CONN_2, P5 CONN_2, P6 CONN_2, Q1 MPSA92, Q2 MPSA42, Q3 MPSA92, Q4 MPSA42, Q5 MPSA92, Q6 MPSA42, Q7 MPSA92, Q8 MPSA42, U1 ICL7660, U2 78L05, U3 LM358N, U4 LM358N

Commit message: Demos update
Connections:
- U1 pad 6: Net-(U1-Pad6) -> unconnected-(U1-Pad6)
- U1 pad 7: Net-(U1-Pad7) -> unconnected-(U1-Pad7)

Commit message: Update demos.
Connections:
- net +12C renamed +12V

Commit message: Demos update.
Connections:
- U1 pad 6: unconnected-(U1-Pad6) -> (no net)
- U1 pad 7: unconnected-(U1-Pad7) -> (no net)
Routing:
- net Net-(R19-Pad2): track 17.2 -> 16.0 mm
- net Net-(D6-Pad1): track 23.0 -> 22.3 mm

Commit message: Demos update
Connections:
- U1 pad 6: (no net) -> unconnected-(U1-Pad6)
- U1 pad 7: (no net) -> unconnected-(U1-Pad7)

Commit message: Demos update.
Parts:
- moved P5 13.8 mm to (181.2, 86.3)
- moved P3 10.5 mm to (181.2, 112.5)
Routing:
- net /ampli_ht_vertical/PIEZO_OUT: track 12.7 -> 16.6 mm
Other:
- board size 100.3 x 80 mm -> 100.7 x 80 mm
Changed lines of the file:
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@@
   )
   (footprint "TerminalBlock_Altech:Altech_AK300_1x02_P5.00mm_45-Degree" (layer "F.Cu")
-    (at 182.245 122.936 90)
+    (at 181.1925 112.4575 90)
     (descr "Altech AK300 serie terminal block (Script generated with StandardBox.py) (http://www.altechcorp.com/PDFS/PCBMETRC.PDF)")
     (tags "Altech AK300 serie connector")
@@
   )
   (footprint "TerminalBlock_Altech:Altech_AK300_1x02_P5.00mm_45-Degree" (layer "F.Cu")
-    (at 182.245 100.076 90)
+    (at 181.2 86.3 90)
     (descr "Altech AK300 serie terminal block (Script generated with StandardBox.py) (http://www.altechcorp.com/PDFS/PCBMETRC.PDF)")
     (tags "Altech AK300 serie connector")
@@
     )
   )
-  (gr_line (start 88.265 131.826) (end 88.265 51.816) (layer "Edge.Cuts") (width 0.2032))
-  (gr_line (start 188.595 131.826) (end 88.265 131.826) (layer "Edge.Cuts") (width 0.2032))
-  (gr_line (start 88.265 51.816) (end 188.595 51.816) (layer "Edge.Cuts") (width 0.2032))
+  (gr_line (start 87.9 131.826) (end 87.9 51.8) (layer "Edge.Cuts") (width 0.2032))
+  (gr_line (start 188.595 131.826) (end 87.9 131.826) (layer "Edge.Cuts") (width 0.2032))
+  (gr_line (start 87.9 51.8) (end 188.595 51.816) (layer "Edge.Cuts") (width 0.2032))
   (gr_line (start 188.595 51.816) (end 188.595 131.826) (layer "Edge.Cuts") (width 0.2032))
   (gr_text "Complex hierarchy\nDemo" (at 177.4 69) (layer "F.Cu")
@@
   (segment (start 95.885 84.836) (end 95.885 83.185) (width 0.4318) (layer "B.Cu") (net 3))
   (segment (start 100.965 80.518) (end 102.743 78.74) (width 0.4318) (layer "B.Cu") (net 3))
-  (segment (start 173.355 100.076) (end 182.245 100.076) (width 0.4318) (layer "B.Cu") (net 4))
+  (segment (start 173.355 89.045) (end 173.355 91.186) (width 0.4) (layer "B.Cu") (net 4))
   (segment (start 173.355 97.536) (end 173.355 91.186) (width 0.4318) (layer "B.Cu") (net 4))
-  (segment (start 173.355 97.536) (end 173.355 100.076) (width 0.4318) (layer "B.Cu") (net 4))
+  (segment (start 176.1 86.3) (end 173.355 89.045) (width 0.4) (layer "B.Cu") (net 4))
+  (segment (start 181.2 86.3) (end 176.1 86.3) (width 0.4) (layer "B.Cu") (net 4))
   (segment (start 116.586 99.187) (end 119.888 99.187) (width 0.4318) (layer "B.Cu") (net 5))
   (segment (start 156.845 89.916) (end 156.845 92.456) (width 0.4318) (layer "B.Cu") (net 5))
@@
   (segment (start 95.758 107.061) (end 102.235 107.061) (width 0.4318) (layer "B.Cu") (net 7))
   (segment (start 173.355 122.936) (end 173.355 119.126) (width 0.4318) (layer "B.Cu") (net 8))
-  (segment (start 173.355 122.936) (end 182.245 122.936) (width 0.4318) (layer "B.Cu") (net 8))
+  (segment (start 173.355 115.445) (end 173.355 119.126) (width 0.4) (layer "B.Cu") (net 8))
+  (segment (start 181.1925 112.4575) (end 176.3425 112.4575) (width 0.4) (layer "B.Cu") (net 8))
+  (segment (start 176.3425 112.4575) (end 173.355 115.445) (width 0.4) (layer "B.Cu") (net 8))
   (segment (start 146.05 120.396) (end 152.4 120.396) (width 0.4318) (layer "B.Cu") (net 9))
   (segment (start 139.319 114.046) (end 139.0015 114.3635) (width 0.4) (layer "B.Cu") (net 9))

Commit message: Demos update
Changed lines of the file:
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@@
     (effects (font (size 2.032 1.524) (thickness 0.3048)))
   )
-  (gr_text "Complex hierarchy\nDemo" (at 176.8 67.2) (layer "B.Cu")
+  (gr_text "Complex hierarchy\nDemo" (at 182 63 90) (layer "B.Cu")
     (effects (font (size 2.032 1.524) (thickness 0.3048)) (justify mirror))
   )
