File: demos/test_xil_95108/carte_test.kicad_sch (KiCad schematic)
At the start: 42 parts, among them J1 DB25, J2 DB9FEM, K1 CONN_3, P2 CONN_3, P3 CONN_2, P4 CONN_2X2, SW1 SW_PUSH, SW2 SW_PUSH, U1 TDA8702, U2 XC95108PC84, U3 LM7805, U4 74HC04, U5 RAM_32KO, U6 LM318N, X1 10MHz

Commit message: Update demos.
Other:
- note added: "Unused"
Changed lines of the file:
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@@
-(kicad_sch (version 20210406) (generator eeschema)
+(kicad_sch (version 20210621) (generator eeschema)
   (paper "A3")
   (title_block
@@
     (stroke (width 0) (type solid) (color 0 0 0 0))
   )
+  (polyline (pts (xy 22.225 239.395) (xy 22.225 281.305))
+    (stroke (width 0) (type default) (color 0 0 0 0))
+  )
+  (polyline (pts (xy 22.225 239.395) (xy 85.09 239.395))
+    (stroke (width 0) (type default) (color 0 0 0 0))
+  )
+  (polyline (pts (xy 85.09 239.395) (xy 85.09 281.305))
+    (stroke (width 0) (type default) (color 0 0 0 0))
+  )
+  (polyline (pts (xy 85.09 281.305) (xy 22.225 281.305))
+    (stroke (width 0) (type default) (color 0 0 0 0))
+  )
+  (text "Unused" (at 67.31 279.4 0)
+    (effects (font (size 1.27 1.27)) (justify left bottom))
+  )
   (label "+12BATT" (at 38.1 198.12 0)
     (effects (font (size 1.524 1.524)) (justify left bottom))
@@
       (effects (font (size 1.524 1.524)))
     )
-    (property "Footprint" "Package_DIP:DIP-14_W7.62mm_LongPads" (id 2) (at 82.55 256.54 0)
-      (effects (font (size 0.508 0.508)))
-    )
+    (property "Footprint" "Package_DIP:DIP-14_W7.62mm_LongPads" (id 2) (at 74.295 256.54 0)
+      (effects (font (size 0.508 0.508)))
+    )

Commit message: Demos update.
Parts:
- J2: footprint Connector_Dsub:DSUB-9_Female_EdgeMount_P2.77mm -> Connector_Dsub:DSUB-9_Female_Horizontal_P2.77x2.84mm_EdgePinOffset4.94mm_Housed_MountingHolesOffset7.48mm

Commit message: Demos update
Parts:
- added U (x2): (no value), symbol carte_test_schlib:-12V
- U: renamed from U1; value TDA8702 -> (none); footprint Package_DIP:DIP-16_W7.62mm_Socket_LongPads -> (none)
- U: renamed from C1; value 100nF -> (none); footprint Capacitors_SMD:C_1206 -> (none)
- U: renamed from C2; value 10uF -> (none); footprint Capacitor_THT:CP_Axial_L10.0mm_D4.5mm_P15.00mm_Horizontal -> (none)
- U: renamed from C3; value 10uF -> (none); footprint Capacitor_THT:CP_Axial_L10.0mm_D4.5mm_P15.00mm_Horizontal -> (none)
- U: renamed from X1; value 10MHz -> (none); footprint Crystal:Crystal_HC18-U_Horizontal -> (none)
- U: renamed from C4; value 22pF -> (none); footprint Capacitors_SMD:C_1206 -> (none)
- U: renamed from R1; value 100K -> (none); footprint Resistor_THT:R_Axial_DIN0207_L6.3mm_D2.5mm_P10.16mm_Horizontal -> (none)
- U: renamed from U3; value LM7805 -> (none); footprint Package_TO_SOT_THT:TO-220-3_Horizontal_TabDown -> (none)
- U: renamed from P2; value CONN_3 -> (none); footprint TerminalBlock_Phoenix:TerminalBlock_Phoenix_MKDS-1,5-3-5.08_1x03_P5.08mm_Horizontal -> (none)
- U: renamed from D1; value 1N4004 -> (none); footprint Diode_THT:D_DO-35_SOD27_P12.70mm_Horizontal -> (none)
- U: renamed from C6; value 47uF -> (none); footprint Capacitor_THT:CP_Axial_L10.0mm_D4.5mm_P15.00mm_Horizontal -> (none)
- U: renamed from P3; value CONN_2 -> (none); footprint TerminalBlock_Phoenix:TerminalBlock_Phoenix_MKDS-1,5-2-5.08_1x02_P5.08mm_Horizontal -> (none)
- U: renamed from U4; value 74HC04 -> (none); footprint Package_DIP:DIP-14_W7.62mm_LongPads -> (none)
- U: renamed from U5; value RAM_32KO -> (none); footprint Sockets_DIP:DIP-28__300__600_ELL -> (none)
- U: renamed from K1; value CONN_3 -> (none); footprint Connector_PinHeader_2.54mm:PinHeader_1x03_P2.54mm_Vertical -> (none)
- U: renamed from J1; value DB25 -> (none); footprint Connector_Dsub:DSUB-25_Female_Horizontal_P2.77x2.84mm_EdgePinOffset9.90mm_Housed_MountingHolesOffset11.32mm -> (none)
- U: renamed from C12; value 100nF -> (none); footprint Capacitors_SMD:C_1206 -> (none)
- U: renamed from R3; value 330 -> (none); footprint Resistor_THT:R_Axial_DIN0207_L6.3mm_D2.5mm_P10.16mm_Horizontal -> (none)
- U: renamed from D3; value LED -> (none); footprint LED_THT:LED_D5.0mm -> (none)
- U: renamed from SW1; value SW_PUSH -> (none); footprint Button_Switch_THT:SW_PUSH_6mm_h4.3mm -> (none)
- U: renamed from SW2; value SW_PUSH -> (none); footprint Button_Switch_THT:SW_PUSH_6mm_h4.3mm -> (none)
- U: renamed from R4; value 4,7K -> (none); footprint Resistor_THT:R_Axial_DIN0207_L6.3mm_D2.5mm_P10.16mm_Horizontal -> (none)
- U: renamed from R5; value 4,7K -> (none); footprint Resistor_THT:R_Axial_DIN0207_L6.3mm_D2.5mm_P10.16mm_Horizontal -> (none)
- U: renamed from P4; value CONN_2X2 -> (none); footprint Connector_PinHeader_2.54mm:PinHeader_2x02_P2.54mm_Vertical -> (none)
- U: renamed from C14; value 10uF -> (none); footprint Capacitor_THT:CP_Axial_L10.0mm_D4.5mm_P15.00mm_Horizontal -> (none)
- U: renamed from R8; value 2,2K -> (none); footprint Resistor_THT:R_Axial_DIN0207_L6.3mm_D2.5mm_P10.16mm_Horizontal -> (none)
- U: renamed from R9; value 2,2K -> (none); footprint Resistor_THT:R_Axial_DIN0207_L6.3mm_D2.5mm_P10.16mm_Horizontal -> (none)
- U: renamed from R6; value 1,1k -> (none); footprint Resistor_THT:R_Axial_DIN0207_L6.3mm_D2.5mm_P10.16mm_Horizontal -> (none)
- U: renamed from R7; value 1,1K -> (none); footprint Resistor_THT:R_Axial_DIN0207_L6.3mm_D2.5mm_P10.16mm_Horizontal -> (none)
- U: renamed from R10; value 75 -> (none); footprint Resistor_THT:R_Axial_DIN0207_L6.3mm_D2.5mm_P10.16mm_Horizontal -> (none)
- U: renamed from U6; value LM318N -> (none); footprint Package_DIP:DIP-8_W7.62mm_LongPads -> (none)
- U: renamed from C13; value 10uF -> (none); footprint Capacitor_THT:CP_Axial_L10.0mm_D4.5mm_P15.00mm_Horizontal -> (none)
- U: renamed from D4; value 1N4004 -> (none); footprint Diode_THT:D_DO-35_SOD27_P12.70mm_Horizontal -> (none)
- U: renamed from J2; value DB9FEM -> (none); footprint Connector_Dsub:DSUB-9_Female_Horizontal_P2.77x2.84mm_EdgePinOffset4.94mm_Housed_MountingHolesOffset7.48mm -> (none)
- U: renamed from C5; value 22pF -> (none); footprint Capacitors_SMD:C_1206 -> (none)
- U: renamed from C11; value 100nF -> (none); footprint Capacitor_SMD:C_1206_3216Metric_Pad1.24x1.80mm_HandSolder -> (none)
- U: renamed from C7; value 100nF -> (none); footprint Capacitor_SMD:C_1206_3216Metric_Pad1.24x1.80mm_HandSolder -> (none)
- U: renamed from C10; value 100nF -> (none); footprint Capacitor_SMD:C_1206_3216Metric_Pad1.24x1.80mm_HandSolder -> (none)
- U: renamed from C8; value 100nF -> (none); footprint Capacitor_SMD:C_1206_3216Metric_Pad1.24x1.80mm_HandSolder -> (none)
- U: renamed from R2; value 330 -> (none); footprint Resistor_THT:R_Axial_DIN0207_L6.3mm_D2.5mm_P10.16mm_Horizontal -> (none)
- U: renamed from D2; value LED -> (none); footprint LED_THT:LED_D5.0mm -> (none)
- U: renamed from U2; value XC95108PC84 -> (none); footprint Sockets:PLCC84 -> (none)
Connections:
- net -12V: now also U.1 (-12V), U.1 (-12V)
- net GND: now also U.1, U.1, U.1, U.1; no longer U.11, U.13, U.5, U.9
- net XIN/CLK: now also U.2; no longer U.4
- net at U.1, U.1, U.2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: now also U.1; no longer U.3

Commit message: Demos update
Connections:
- net GND: now also U.11, U.13, U.5, U.9; no longer U.1, U.1, U.1, U.1
- net XIN/CLK: now also U.4; no longer U.2
- net at U.1, U.1, U.2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: now also U.3; no longer U.1
Changed lines of the file:
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@@
-(kicad_sch (version 20220404) (generator eeschema)
+(kicad_sch (version 20220822) (generator eeschema)
   (paper "A3")
   (title_block
@@
     (pin "1")
     (pin "2")
+  )
+  (symbol (lib_id "carte_test_schlib:74HC04") (at 173.99 226.06 0) (unit 2)
+    (in_bom yes) (on_board yes)
+    (default_instance (reference "U") (unit 1) (value "") (footprint ""))
+    (property "Reference" "U" (id 0) (at 178.943 223.139 0)
+      (effects (font (size 1.524 1.524)))
+    )
+    (property "Value" "" (id 1) (at 178.816 229.2096 0)
+      (effects (font (size 1.524 1.524)))
+    )
+    (property "Footprint" "" (id 2) (at 180.34 231.14 0)
+      (effects (font (size 0.508 0.508)))
+    )
+    (property "Datasheet" "" (id 3) (at 173.99 226.06 0)
+      (effects (font (size 1.524 1.524)) hide)
+    )
+    (pin "14")
+    (pin "7")
     (pin "3")
     (pin "4")
+  )
+  (symbol (lib_id "carte_test_schlib:74HC04") (at 39.37 247.65 0) (unit 3)
+    (in_bom yes) (on_board yes)
+    (default_instance (reference "U") (unit 1) (value "") (footprint ""))
+    (property "Reference" "U" (id 0) (at 44.323 244.729 0)
+      (effects (font (size 1.524 1.524)))
+    )
+    (property "Value" "" (id 1) (at 44.196 250.7996 0)
+      (effects (font (size 1.524 1.524)))
+    )
+    (property "Footprint" "" (id 2) (at 39.37 241.3 0)
+      (effects (font (size 0.508 0.508)))
+    )
+    (property "Datasheet" "" (id 3) (at 39.37 247.65 0)
+      (effects (font (size 1.524 1.524)) hide)
+    )
+    (pin "14")
+    (pin "7")
     (pin "5")
     (pin "6")
+  )
+  (symbol (lib_id "carte_test_schlib:74HC04") (at 39.37 261.62 0) (unit 4)
+    (in_bom yes) (on_board yes)
+    (default_instance (reference "U") (unit 1) (value "") (footprint ""))
+    (property "Reference" "U" (id 0) (at 44.323 258.699 0)
+      (effects (font (size 1.524 1.524)))
+    )
+    (property "Value" "" (id 1) (at 44.196 264.7696 0)
+      (effects (font (size 1.524 1.524)))
+    )
+    (property "Footprint" "" (id 2) (at 45.72 256.54 0)
+      (effects (font (size 0.508 0.508)))
+    )
+    (property "Datasheet" "" (id 3) (at 39.37 261.62 0)
+      (effects (font (size 1.524 1.524)) hide)
+    )
+    (pin "14")
+    (pin "7")
     (pin "8")
     (pin "9")
+  )
+  (symbol (lib_id "carte_test_schlib:74HC04") (at 39.37 274.32 0) (unit 5)
+    (in_bom yes) (on_board yes)
+    (default_instance (reference "U") (unit 1) (value "") (footprint ""))
+    (property "Reference" "U" (id 0) (at 44.323 271.399 0)
+      (effects (font (size 1.524 1.524)))
+    )
+    (property "Value" "" (id 1) (at 44.196 277.4696 0)
+      (effects (font (size 1.524 1.524)))
+    )
+    (property "Footprint" "" (id 2) (at 48.26 269.24 0)
+      (effects (font (size 0.508 0.508)))
+    )
+    (property "Datasheet" "" (id 3) (at 39.37 274.32 0)
+      (effects (font (size 1.524 1.524)) hide)
+    )
+    (pin "14")
+    (pin "7")
     (pin "10")
     (pin "11")
+  )
+  (symbol (lib_id "carte_test_schlib:74HC04") (at 67.31 261.62 0) (unit 6)
+    (in_bom yes) (on_board yes)
+    (default_instance (reference "U") (unit 1) (value "") (footprint ""))
+    (property "Reference" "U" (id 0) (at 72.263 258.699 0)
+      (effects (font (size 1.524 1.524)))
+    )
+    (property "Value" "" (id 1) (at 72.136 264.7696 0)
+      (effects (font (size 1.524 1.524)))
+    )
+    (property "Footprint" "" (id 2) (at 74.295 256.54 0)
+      (effects (font (size 0.508 0.508)))
+    )
+    (property "Datasheet" "" (id 3) (at 67.31 261.62 0)
+      (effects (font (size 1.524 1.524)) hide)
+    )
+    (pin "14")
+    (pin "7")
     (pin "12")
     (pin "13")
-  )
-  (symbol (lib_id "carte_test_schlib:74HC04") (at 173.99 226.06 0) (unit 1)
-    (in_bom yes) (on_board yes)
-    (default_instance (reference "U") (unit 1) (value "") (footprint ""))
-    (property "Reference" "U" (id 0) (at 178.943 223.139 0)
-      (effects (font (size 1.524 1.524)))
-    )
-    (property "Value" "" (id 1) (at 178.816 229.2096 0)
-      (effects (font (size 1.524 1.524)))
-    )
-    (property "Footprint" "" (id 2) (at 180.34 231.14 0)
-      (effects (font (size 0.508 0.508)))
-    )
-    (property "Datasheet" "" (id 3) (at 173.99 226.06 0)
-      (effects (font (size 1.524 1.524)) hide)
-    )
-    (pin "14")
-    (pin "7")
-    (pin "1")
-    (pin "2")
-    (pin "3")
-    (pin "4")
-    (pin "5")
-    (pin "6")
-    (pin "8")
-    (pin "9")
-    (pin "10")
-    (pin "11")
-    (pin "12")
-    (pin "13")
-  )
-  (symbol (lib_id "carte_test_schlib:74HC04") (at 39.37 247.65 0) (unit 1)
-    (in_bom yes) (on_board yes)
-    (default_instance (reference "U") (unit 1) (value "") (footprint ""))
-    (property "Reference" "U" (id 0) (at 44.323 244.729 0)
-      (effects (font (size 1.524 1.524)))
-    )
-    (property "Value" "" (id 1) (at 44.196 250.7996 0)
-      (effects (font (size 1.524 1.524)))
-    )
-    (property "Footprint" "" (id 2) (at 39.37 241.3 0)
-      (effects (font (size 0.508 0.508)))
-    )
-    (property "Datasheet" "" (id 3) (at 39.37 247.65 0)
-      (effects (font (size 1.524 1.524)) hide)
-    )
-    (pin "14")
-    (pin "7")
-    (pin "1")
-    (pin "2")
-    (pin "3")
-    (pin "4")
-    (pin "5")
-    (pin "6")
-    (pin "8")
-    (pin "9")
-    (pin "10")
-    (pin "11")
-    (pin "12")
-    (pin "13")
-  )
-  (symbol (lib_id "carte_test_schlib:74HC04") (at 39.37 261.62 0) (unit 1)
-    (in_bom yes) (on_board yes)
-    (default_instance (reference "U") (unit 1) (value "") (footprint ""))
-    (property "Reference" "U" (id 0) (at 44.323 258.699 0)
-      (effects (font (size 1.524 1.524)))
-    )
-    (property "Value" "" (id 1) (at 44.196 264.7696 0)
-      (effects (font (size 1.524 1.524)))
-    )
-    (property "Footprint" "" (id 2) (at 45.72 256.54 0)
-      (effects (font (size 0.508 0.508)))
-    )
-    (property "Datasheet" "" (id 3) (at 39.37 261.62 0)
-      (effects (font (size 1.524 1.524)) hide)
-    )
-    (pin "14")
-    (pin "7")
-    (pin "1")
-    (pin "2")
-    (pin "3")
-    (pin "4")
-    (pin "5")
-    (pin "6")
-    (pin "8")
-    (pin "9")
-    (pin "10")
-    (pin "11")
-    (pin "12")
-    (pin "13")
-  )
-  (symbol (lib_id "carte_test_schlib:74HC04") (at 39.37 274.32 0) (unit 1)
-    (in_bom yes) (on_board yes)
-    (default_instance (reference "U") (unit 1) (value "") (footprint ""))
-    (property "Reference" "U" (id 0) (at 44.323 271.399 0)
-      (effects (font (size 1.524 1.524)))
-    )
-    (property "Value" "" (id 1) (at 44.196 277.4696 0)
-      (effects (font (size 1.524 1.524)))
-    )
-    (property "Footprint" "" (id 2) (at 48.26 269.24 0)
-      (effects (font (size 0.508 0.508)))
-    )
-    (property "Datasheet" "" (id 3) (at 39.37 274.32 0)
-      (effects (font (size 1.524 1.524)) hide)
-    )
-    (pin "14")
-    (pin "7")
-    (pin "1")
-    (pin "2")
-    (pin "3")
-    (pin "4")
-    (pin "5")
-    (pin "6")
-    (pin "8")
-    (pin "9")
-    (pin "10")
-    (pin "11")
-    (pin "12")
-    (pin "13")
-  )
-  (symbol (lib_id "carte_test_schlib:74HC04") (at 67.31 261.62 0) (unit 1)
-    (in_bom yes) (on_board yes)
-    (default_instance (reference "U") (unit 1) (value "") (footprint ""))
-    (property "Reference" "U" (id 0) (at 72.263 258.699 0)
-      (effects (font (size 1.524 1.524)))
-    )
-    (property "Value" "" (id 1) (at 72.136 264.7696 0)
-      (effects (font (size 1.524 1.524)))
-    )
-    (property "Footprint" "" (id 2) (at 74.295 256.54 0)
-      (effects (font (size 0.508 0.508)))
-    )
-    (property "Datasheet" "" (id 3) (at 67.31 261.62 0)
-      (effects (font (size 1.524 1.524)) hide)
-    )
-    (pin "14")
-    (pin "7")
-    (pin "1")
-    (pin "2")
-    (pin "3")
-    (pin "4")
-    (pin "5")
-    (pin "6")
-    (pin "8")
-    (pin "9")
-    (pin "10")
-    (pin "11")
-    (pin "12")
-    (pin "13")
