File: qa/data/pcbnew/issue18.kicad_pcb (KiCad board)
At the start: 6 copper layers, 1 part, among them U13 TestFootprint

Commit message: Update qa tests to use new zone fill algo
Other:
- net class Default removed
