File: qa/data/pcbnew/issue5102.kicad_pcb (KiCad board)
At the start: 4 copper layers, 100 x 64 mm, 92 parts, among them IC1 24C01, P1 FE04-1, P10 JSTPHMHS-2, P2 MA07-2S-1.27, P3 JSTPHMHS-2, P4 FE04-1, P5 FE02-1, P8 USB_B, Q1 BSS138, Q2 BSS138, Q3 BSS138, Q4 BSS138, SW1 SK12D07-G8, U1 STM32L151C8Tx, U2 LM4132AMF-4.1, U3 MAX5217GUA+, U4 OPA333AIDCKR, U5 TPS61085, U6 TP4056, U7 HT7833, U8 HT7850, U9 LM2776

Commit message: Update qa tests to use new zone fill algo
Routing:
- added copper zone on In2.Cu, net /3V3
- added copper zone on In2.Cu, net /5V
- added copper zone on In2.Cu, net /5VFILT
- added copper zone on In1.Cu, net GND
- added copper zone on In1.Cu, net GNDA
- removed copper zone on PWR, net /3V3
- removed copper zone on PWR, net /5V
- removed copper zone on PWR, net /5VFILT
- removed copper zone on GND, net GND
- removed copper zone on GND, net GNDA
