File: qa/data/pcbnew/issue6284.kicad_pcb (KiCad board)
At the start: 2 copper layers, 160 x 100 mm, 134 parts, among them P101 DIN41612_M_3x32_OS2, U101 2MHz, U102 'HC161, U103 'HC161, U104 'HC161, U105 'HC161, U106 'HC14, U107 'HC10, U108 'HC109, U109 'HC02, U110 NE5532, U111 'HC245, U112 NE5532, U113 'HC86, U114 'HC109, U115 'HC109, U116 'HCT273, U117 'HCT273, U118 'HC10, U119 'HC03, U120 'HC237, U121 27C512

Commit message: Update qa tests to use new zone fill algo
Connections:
- net /Circuit/~LASTDOT renamed /Circuit/~{LASTDOT}
- net /Circuit/~LASTLINE renamed /Circuit/~{LASTLINE}
- net /Circuit/~LASTPOSREQ renamed /Circuit/~{LASTPOSREQ}
