File: demos/jetson-agx-thor-baseboard/expansion_connector.kicad_sch (KiCad schematic)
At the start: 38 parts, among them J18 ASP-218650-01_mounting_holes, J8 Plug_Samtec_UMPT_1x6_UMPT-06-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, U2 AT24CS01_SOIC8

Commit message: Update Antmicro Jetson Thor board
Per request, updating the schematc/board and README
Other:
- title: Jetson AGX Thor Baseboard -> Antmicro Baseboard for Jetson AGX Thor
Changed lines of the file:
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@@
 	(paper "A3")
 	(title_block
-		(title "Jetson AGX Thor Baseboard")
-		(date "2025-11-03")
+		(title "Antmicro Baseboard for Jetson AGX Thor")
+		(date "2026-02-17")
 		(rev "1.1.0")
 		(company "Antmicro Ltd")
@@
 		(polyline
 			(pts
-				(xy 251.46 255.27) (xy 288.29 255.27) (xy 288.29 203.2) (xy 251.46 203.2)
+				(xy 173.99 247.65) (xy 210.82 247.65) (xy 210.82 215.9) (xy 173.99 215.9)
 			)
 			(stroke
@@
 		(polyline
 			(pts
-				(xy 173.99 247.65) (xy 210.82 247.65) (xy 210.82 215.9) (xy 173.99 215.9)
+				(xy 251.46 255.27) (xy 288.29 255.27) (xy 288.29 203.2) (xy 251.46 203.2)
 			)
 			(stroke
