File: demos/jetson-agx-thor-baseboard/power.kicad_sch (KiCad schematic)
At the start: 76 parts, among them J2 Molex_Mini-Fit_2x3_50362462, Q16 DMG1012T-7, Q2 SISS05DN-T1-GE3, Q23 SISS05DN-T1-GE3, Q24 SISS05DN-T1-GE3, Q25 SISS05DN-T1-GE3, Q39 SISS05DN-T1-GE3, Q4 DMG1012T-7, Q5 SISS05DN-T1-GE3, Q6 DMG1012T-7, Q9 SISS05DN-T1-GE3, U15 NCP718BSN330T1G, U6 LTC4412IS6, U61 LTC4412IS6, U62 LTC4412IS6, U63 LTC4412IS6, U64 LTC4412IS6

Commit message: Update Antmicro Jetson Thor board
Per request, updating the schematc/board and README
Other:
- title: Jetson AGX Thor Baseboard -> Antmicro Baseboard for Jetson AGX Thor
Changed lines of the file:
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@@
 	(paper "A3")
 	(title_block
-		(title "Jetson AGX Thor Baseboard")
-		(date "2025-11-03")
+		(title "Antmicro Baseboard for Jetson AGX Thor")
+		(date "2026-02-17")
 		(rev "1.1.0")
 		(company "Antmicro Ltd")
