File: demos/jetson-agx-thor-baseboard/recovery_usb.kicad_sch (KiCad schematic)
At the start: 49 parts, among them J3 USB-C_Kycon_KUSBX-SL2-CS1N24-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, Q15 DMG1012T-7, Q19 DMG1012T-7, U23 AP22615A_TSOT26, U26 TPD4E05U06QDQARQ1, U56 HD3SS3220IRNHR, U57 TPD4E05U06QDQARQ1, U58 TPD4E05U06QDQARQ1

Commit message: Update Antmicro Jetson Thor board
Per request, updating the schematc/board and README
Other:
- title: Jetson AGX Thor Baseboard -> Antmicro Baseboard for Jetson AGX Thor
Changed lines of the file:
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@@
 	(paper "A3")
 	(title_block
-		(title "Jetson AGX Thor Baseboard")
-		(date "2025-11-03")
+		(title "Antmicro Baseboard for Jetson AGX Thor")
+		(date "2026-02-17")
 		(rev "1.1.0")
 		(company "Antmicro Ltd")
@@
 		(polyline
 			(pts
-				(xy 158.75 165.1) (xy 110.49 165.1) (xy 110.49 149.86) (xy 158.75 149.86)
+				(xy 281.305 147.955) (xy 269.24 147.955) (xy 269.24 142.24) (xy 281.305 142.24)
 			)
 			(stroke
@@
 		(polyline
 			(pts
-				(xy 248.92 180.975) (xy 189.3887 180.975) (xy 189.23 149.86) (xy 248.92 149.86)
+				(xy 158.75 165.1) (xy 110.49 165.1) (xy 110.49 149.86) (xy 158.75 149.86)
 			)
 			(stroke
@@
 		(polyline
 			(pts
-				(xy 281.305 147.955) (xy 269.24 147.955) (xy 269.24 142.24) (xy 281.305 142.24)
+				(xy 248.92 180.975) (xy 189.3887 180.975) (xy 189.23 149.86) (xy 248.92 149.86)
 			)
 			(stroke
