File: demos/jetson-agx-thor-baseboard/sfp.kicad_sch (KiCad schematic)
At the start: 35 parts, among them J12 Amphenol_SFP28_1x20_UE763GA20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, J19 Amphenol_SFP28_Cage_U773GC163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, U73 TPD4E05U06QDQARQ1

Commit message: Update Antmicro Jetson Thor board
Per request, updating the schematc/board and README
Other:
- title: Jetson AGX Thor Baseboard -> Antmicro Baseboard for Jetson AGX Thor
Changed lines of the file:
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@@
 	(paper "A3")
 	(title_block
-		(title "Jetson AGX Thor Baseboard")
-		(date "2025-11-03")
+		(title "Antmicro Baseboard for Jetson AGX Thor")
+		(date "2026-02-17")
 		(rev "1.1.0")
 		(company "Antmicro Ltd")
