File: demos/jetson-agx-thor-baseboard/usb_hub.kicad_sch (KiCad schematic)
At the start: 131 parts, among them J5 USB-C_Kycon_KUSBX-SL2-CS1N24-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, J6 USB-C_Kycon_KUSBX-SL2-CS1N24-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, Q21 DMC2400UV-7, Q26 DMC2400UV-7, Q27 DMC2400UV-7, Q29 DMC2400UV-7, U17 TPD4E05U06QDQARQ1, U18 AP22615A_TSOT26, U19 TPD4E05U06QDQARQ1, U20 AP22615A_TSOT26, U21 USB7252C, U24 TPD4E05U06QDQARQ1, U25 TPD4E05U06QDQARQ1, U27 TPD4E05U06QDQARQ1, U28 TPD4E05U06QDQARQ1, U52 SST26VF064B, Y2 Oscillator_25MHz_ESC_2016MV

Commit message: Update Antmicro Jetson Thor board
Per request, updating the schematc/board and README
Other:
- title: Jetson AGX Thor Baseboard -> Antmicro Baseboard for Jetson AGX Thor
Changed lines of the file:
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@@
 	(paper "A3")
 	(title_block
-		(title "Jetson AGX Thor Baseboard")
-		(date "2025-11-03")
+		(title "Antmicro Baseboard for Jetson AGX Thor")
+		(date "2026-02-17")
 		(rev "1.1.0")
 		(company "Antmicro Ltd")
@@
 		(polyline
 			(pts
-				(xy 313.5312 231.14) (xy 259.2387 231.14) (xy 259.08 200.66) (xy 313.3725 200.66)
+				(xy 313.5312 109.22) (xy 259.2387 109.22) (xy 259.08 78.74) (xy 313.3725 78.74)
 			)
 			(stroke
@@
 		(polyline
 			(pts
-				(xy 313.5312 109.22) (xy 259.2387 109.22) (xy 259.08 78.74) (xy 313.3725 78.74)
+				(xy 123.19 89.535) (xy 73.66 89.535) (xy 73.66 83.185) (xy 123.19 83.185)
 			)
 			(stroke
@@
 		(polyline
 			(pts
-				(xy 271.145 193.675) (xy 259.08 193.675) (xy 259.08 187.96) (xy 271.145 187.96)
+				(xy 313.5312 231.14) (xy 259.2387 231.14) (xy 259.08 200.66) (xy 313.3725 200.66)
 			)
 			(stroke
@@
 		(polyline
 			(pts
-				(xy 123.19 89.535) (xy 73.66 89.535) (xy 73.66 83.185) (xy 123.19 83.185)
+				(xy 271.145 71.755) (xy 259.08 71.755) (xy 259.08 66.04) (xy 271.145 66.04)
 			)
 			(stroke
@@
 		(polyline
 			(pts
-				(xy 271.145 71.755) (xy 259.08 71.755) (xy 259.08 66.04) (xy 271.145 66.04)
+				(xy 271.145 193.675) (xy 259.08 193.675) (xy 259.08 187.96) (xy 271.145 187.96)
 			)
 			(stroke
