File: qa/data/eeschema/api_kitchen_sink.kicad_sch (KiCad schematic)
At the start: 3 parts, among them Q1 Q_NPN, U1 STM32C011J_4-6_Mx

Commit message: API: expand symbol support
Also fix textbox not using border_enabled
Parts:
- added R2: JUMPER, symbol Device:R_US
- added R3: PASSTHROUGH, symbol Device:R
Connections:
- net at U1.7 (PA13): now also R3.2
- net at U1.8 (PA14/PB6/PC15): now also R2.2
- net at Q1.C: now also R2.1
- net at Q1.E: now also R3.1
